File: LoRa-device.kicad_pcb (KiCad board)
At the start: 4 copper layers, 86.4 x 50.8 mm, 128 parts, among them J1 Connector, USB-TYPE-C-16P, J2 Conn_01x02_Pin, J3 Conn_Coaxial, J4 Conn_01x14_Pin, J6 Conn_01x04_Pin, J7 Screw_Terminal_01x08, J8 U.FL, Q2 S8050, SW2 SW_DPST_x2, U1 ESP32-S3, U10 TPS2116DRL, U11 L76KB-A58, U13 MCP23S17_ML, U2 W25Q128JVS, U3 TP4055, U4 ATECC608A-SSHDA, U5 Ai-Thinker-Ra-01, U6 USBLC6-2P6, U7 STLQ015M33R, U8 TPS22917LDBV, U9 AP63203WU, Y1 32.768 kHz, Y2 40MHz(10ppm)

Commit message: Major overhaul of version A
Parts:
- removed C30: 1uF, PCM_JLCPCB:C_0402
- removed J7: Screw_Terminal_01x08, Connector_Phoenix_MC:PhoenixContact_MC_1,5_8-G-3.81_1x08_P3.81mm_Horizontal
- removed R14, R17: 5.1K, Resistor_SMD:R_0402_1005Metric
- removed R37: 4.7kΩ, PCM_JLCPCB:R_0402
- removed R40: 100kΩ, PCM_JLCPCB:R_0402
- removed R41: 47Ω, PCM_JLCPCB:R_0402
- removed R42, R43, R44, R45, R46: 100Ω, PCM_JLCPCB:R_0402
- removed TP1, TP2: TestPoint_2Pole, TestPoint:TestPoint_2Pads_Pitch2.54mm_Drill0.8mm
- added C43: 0.1uF, Capacitor_SMD:C_0402_1005Metric, F.Cu at (132.2, 106.8)
- added MK1: SPH0645LM4H, Sensor_Audio:Knowles_SPH0645LM4H-6_3.5x2.65mm, F.Cu at (139.3, 121.8)
- added R1: 10K, Resistor_SMD:R_0402_1005Metric, F.Cu at (132.2, 105.2)
- added R33: 8.2kΩ, PCM_JLCPCB:R_0402, F.Cu at (118.2, 102.3)
- added R34: 5.1K, Resistor_SMD:R_0402_1005Metric, F.Cu at (127.4, 114.8)
- G***: moved to B.Cu
- J1: value Connector, USB-TYPE-C-16P -> Micro_SD_Card_Det1; footprint PCM_JLCPCB:TYPE-C-SMD_HX-TYPE-C-16PIN -> Lora-device:TF-SMD_TF-01A
- J3: footprint Connector_Coaxial:SMA_Molex_73251-1153_EdgeMount_Horizontal -> Lora-device:SMA-SMD_BWSMA-KE-P001
- R32: value 100K -> 100kΩ; footprint Resistor_SMD:R_0402_1005Metric -> PCM_JLCPCB:R_0402
- R35: value 4.7kΩ -> 5.1K; footprint PCM_JLCPCB:R_0402 -> Resistor_SMD:R_0402_1005Metric
- R4: value 4.7kΩ -> 10K; footprint PCM_JLCPCB:R_0402 -> Resistor_SMD:R_0402_1005Metric
- R6: value 4.7kΩ -> 22kΩ
- U4: value ATECC608A-SSHDA -> MC-121-L119; footprint Package_SO:SOIC-8_3.9x4.9mm_P1.27mm -> Lora-device:USB-C-SMD_HANBO_MC-121-L119
- moved J1 56.2 mm to (172.3, 84.3), turned to 180 degrees
- moved U13 55.5 mm to (136.3, 110.5)
- moved R35 46.6 mm to (131.2, 114.9), turned to -90 degrees
- moved RESET1 43.3 mm to (183.5, 114.4), turned to 0 degrees
- moved J3 43.1 mm to (174.4, 121.7)
- moved J8 42.9 mm to (159.1, 77.3), turned to 90 degrees
- moved FLASH1 42.6 mm to (183.6, 110.6), turned to 0 degrees
- moved R22 38.6 mm to (179.9, 115.4), turned to -90 degrees
- moved C15 38.0 mm to (179.9, 113.4), turned to 90 degrees
- moved R21 37.3 mm to (179.9, 109.6), turned to 90 degrees
- moved L4 36.9 mm to (156.9, 83.1), turned to -90 degrees
- moved DNP4 36.5 mm to (163.3, 121.7), turned to 180 degrees
- moved DNP7 36.4 mm to (160.9, 84.2), turned to 0 degrees
- moved C27 35.2 mm to (158.3, 84.5), turned to 90 degrees
- moved DNP6 34.5 mm to (160.9, 85.5), turned to 0 degrees
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Connections:
- D3 pad 2: IO1 -> GPA5
- J6 pad 1: SD_CS -> unconnected-(J6-Pin_1-Pad1)
- J6 pad 2: MOSIA -> unconnected-(J6-Pin_2-Pad2)
- J6 pad 3: Net-(J6-Pin_3) -> unconnected-(J6-Pin_3-Pad3)
- J6 pad 4: SCKA -> unconnected-(J6-Pin_4-Pad4)
- R10 pad 2: LORA_CS -> SPICLK_N/IO48/LORA_CS
- R24 pad 2: TX -> U0TXD/IO43
- R32 pad 1: GND -> GPA6
- R35 pad 1: VDD_CPU -> GND
- R35 pad 2: Net-(J7-Pin_7) -> Net-(U4-CC2)
- R4 pad 2: SE_SCL -> EXP_RST
- R6 pad 1: VDD_CPU -> +5V
- R6 pad 2: SE_SDA -> Net-(U10-PR1)
- U1 pad 12: IO7 -> GPS_1PPS
- U1 pad 13: GPS_WKUP -> IO8
- U1 pad 15: SCREEN_CS -> IO10
- U1 pad 23: SCREEN_RST -> IO17
- U1 pad 24: TOUCH_CS -> IO18
- U1 pad 36: SE_SCL -> SPICLK_N/IO48/LORA_CS
- U1 pad 37: SE_SDA -> SPICLK_P/IO47/EXP_CS
- U1 pad 38: IO33 -> unconnected-(U1-GPIO33-Pad38)
- U1 pad 39: LORA_CS -> unconnected-(U1-GPIO34-Pad39)
- U1 pad 40: SD_CS -> unconnected-(U1-GPIO35-Pad40)
- U1 pad 41: LORA_IO1 -> unconnected-(U1-GPIO36-Pad41)
- U1 pad 42: LORA_RST -> unconnected-(U1-GPIO37-Pad42)
- U1 pad 50: RX -> U0RXD/IO44
- U1 pad 9: GPS_RST -> IO4
- U10 pad 4: +5V -> Net-(U10-PR1)
- U10 pad 8: unconnected-(U10-ST-Pad8) -> GPA6
- U11 pad 4: unconnected-(U11-1PPS-Pad4) -> GPS_1PPS
- U13 pad 1: unconnected-(U13-GPB4-Pad1) -> SCREEN_CS
- U13 pad 10: unconnected-(U13-SO-Pad10) -> MISOB
- U13 pad 11: unconnected-(U13-A0-Pad11) -> GND
- U13 pad 12: unconnected-(U13-A1-Pad12) -> GND
- U13 pad 13: unconnected-(U13-A2-Pad13) -> GND
- U13 pad 14: unconnected-(U13-~{RESET}-Pad14) -> EXP_RST
- U13 pad 15: unconnected-(U13-INTB-Pad15) -> IO18
- U13 pad 16: unconnected-(U13-INTA-Pad16) -> IO10
- U13 pad 17: unconnected-(U13-GPA0-Pad17) -> LORA_RST
- U13 pad 18: unconnected-(U13-GPA1-Pad18) -> LORA_IO1
- U13 pad 19: unconnected-(U13-GPA2-Pad19) -> SCREEN_RST
- U13 pad 2: unconnected-(U13-GPB5-Pad2) -> TOUCH_CS
- U13 pad 20: unconnected-(U13-GPA3-Pad20) -> GPS_RST
- U13 pad 21: unconnected-(U13-GPA4-Pad21) -> GPS_WKUP
- U13 pad 22: unconnected-(U13-GPA5-Pad22) -> GPA5
- U13 pad 23: unconnected-(U13-GPA6-Pad23) -> GPA6
- U13 pad 24: unconnected-(U13-GPA7-Pad24) -> SD_CS
- U13 pad 25: unconnected-(U13-GPB0-Pad25) -> LORA_IO2
- U13 pad 26: unconnected-(U13-GPB1-Pad26) -> LORA_IO3
- U13 pad 27: unconnected-(U13-GPB2-Pad27) -> LORA_IO4
- U13 pad 28: unconnected-(U13-GPB3-Pad28) -> LORA_IO5
- U13 pad 29: unconnected-(U13-EP-Pad29) -> GND
- U13 pad 3: unconnected-(U13-GPB6-Pad3) -> GPB6
- U13 pad 4: unconnected-(U13-GPB7-Pad4) -> GPB7
- U13 pad 5: unconnected-(U13-VDD-Pad5) -> VDD_CPU
- U13 pad 6: unconnected-(U13-VSS-Pad6) -> GND
- U13 pad 7: unconnected-(U13-~{CS}-Pad7) -> SPICLK_P/IO47/EXP_CS
- U13 pad 8: unconnected-(U13-SCK-Pad8) -> SCKB
- U13 pad 9: unconnected-(U13-SI-Pad9) -> MOSIB
- U5 pad 10: Net-(U5-DIO4) -> LORA_IO4
- U5 pad 11: Net-(U5-DIO5) -> LORA_IO5
- U5 pad 15: LORA_CS -> SPICLK_N/IO48/LORA_CS
- U5 pad 7: unconnected-(U5-DIO2-Pad7) -> LORA_IO2
- U5 pad 8: unconnected-(U5-DIO3-Pad8) -> LORA_IO3
- U6 pad 1: Net-(J1-D--PadA7) -> Net-(U4-DN1)
- U6 pad 3: Net-(J1-D+-PadA6) -> Net-(U4-DP1)
Routing:
- net VDD_CPU: track 339.5 -> 1.56 mm, vias 10 -> 0
- net IO7: track 78.9 -> 0.00 mm, vias 2 -> 0
- net Net-(SW2A-B): track 88.2 -> 19.2 mm, vias 2 -> 1
- net GPS_WKUP: track 63.3 -> 0.00 mm, vias 2 -> 0
- net SCKA: track 79.6 -> 16.5 mm, vias 4 -> 2
- net IO33: track 62.2 -> 0.00 mm, vias 2 -> 0
- net MOSIA: track 74.7 -> 12.7 mm, vias 3 -> 1
- net MISOA: track 80.1 -> 19.8 mm, vias 5 -> 2
- net GPS_RST: track 59.5 -> 0.00 mm, vias 2 -> 0
- net BUZZER: track 70.6 -> 14.2 mm, vias 2 -> 0
- net SD_CS: track 59.1 -> 4.12 mm, vias 1 -> 0
- net LORA_CS: track 47.7 -> 0.00 mm, vias 2 -> 0
- net LORA_RST: track 36.8 -> 0.00 mm
- net IO8: track 0.00 -> 36.7 mm, vias 0 -> 1
- net GPS_1PPS: track 0.00 -> 36.1 mm, vias 0 -> 1
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- added copper zone on In2.Cu, net VDD_CPU
- removed copper zone on In2.Cu, net GND
Other:
- board text removed: "3.3V 3.3V GND SCK MISO MOSI IO5 IO11"
- board text removed: "CLK MISO MOSI CS"
- board text removed: "ILI9341"
- board text removed: "SD"

Commit message: Just a backup.
Parts:
- removed J3: Conn_Coaxial, Lora-device:SMA-SMD_BWSMA-KE-P001
- removed MK1: SPH0645LM4H, Sensor_Audio:Knowles_SPH0645LM4H-6_3.5x2.65mm
- added C30: 100nF, PCM_JLCPCB:C_0402, F.Cu at (161.2, 105.7)
- added C44: 220pF, PCM_JLCPCB:C_0402, F.Cu at (161.2, 107.5)
- added C45: 1uF, PCM_JLCPCB:C_0402, F.Cu at (161.2, 109.4)
- added J5: Conn_01x07_Pin, Connector_PinSocket_2.54mm:PinSocket_1x07_P2.54mm_Horizontal, F.Cu at (164.5, 118.8)
- added R14: 10K, Resistor_SMD:R_0402_1005Metric, F.Cu at (165.7, 96.9)
- added R17: 10K, Resistor_SMD:R_0402_1005Metric, F.Cu at (165.7, 98.9)
- added R37: 10K, Resistor_SMD:R_0402_1005Metric, F.Cu at (165.7, 100.9)
- added R38: 33Ω, PCM_JLCPCB:R_0805, F.Cu at (162.0, 97.4)
- added R39: 33Ω, PCM_JLCPCB:R_0805, F.Cu at (162.0, 100.3)
- added R40: 33Ω, PCM_JLCPCB:R_0805, F.Cu at (162.0, 103.3)
- added R41: 4.7kΩ, PCM_JLCPCB:R_0402, F.Cu at (164.6, 106.3)
- added R42: 4.7kΩ, PCM_JLCPCB:R_0402, F.Cu at (164.6, 108.2)
- added SW1: CK_KMS2xxGP, Button_Switch_SMD:SW_SPST_CK_KMS2xxGP, F.Cu at (153.4, 122.3)
- added SW3: CK_KMS2xxGP, Button_Switch_SMD:SW_SPST_CK_KMS2xxGP, F.Cu at (147.2, 122.3)
- moved DNP2 3.58 mm to (161.1, 115.7)
- moved DNP4 3.58 mm to (160.1, 120.1)
- moved L1 3.58 mm to (160.6, 117.9)
- moved U5 3.58 mm to (150.6, 110.3)
- moved C36 3.58 mm to (162.1, 112.5)
- moved C7 3.58 mm to (161.4, 111.9)
- moved U7 3.43 mm to (148.6, 92.2)
- moved C20 3.43 mm to (149.8, 88.4)
- moved C23 3.43 mm to (149.8, 87.4)
- moved C24 3.43 mm to (149.8, 86.4)
- moved C34 3.43 mm to (148.1, 89.7)
- moved C41 3.43 mm to (148.1, 95.0)
- moved C28 2.71 mm to (156.4, 82.5)
- moved C29 2.71 mm to (156.4, 83.5)
- moved DNP7 2.71 mm to (161.7, 81.5)
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Connections:
- J1 pad 1: unconnected-(J1-DAT2-Pad1) -> Net-(J1-DAT2)
- J1 pad 10: unconnected-(J1-SHIELD-Pad10) -> GND
- J1 pad 2: unconnected-(J1-DAT3/CD-Pad2) -> SD_CS
- J1 pad 3: unconnected-(J1-CMD-Pad3) -> MOSIA
- J1 pad 4: unconnected-(J1-VDD-Pad4) -> VDD_CPU
- J1 pad 5: unconnected-(J1-CLK-Pad5) -> SCKA
- J1 pad 6: unconnected-(J1-VSS-Pad6) -> GND
- J1 pad 7: unconnected-(J1-DAT0-Pad7) -> MISOA
- J1 pad 8: unconnected-(J1-DAT1-Pad8) -> Net-(J1-DAT1)
- J1 pad 9: unconnected-(J1-DET-Pad9) -> GPB6
- U1 pad 6: IO1 -> Net-(U1-GPIO1)
- U1 pad 9: IO4 -> Net-(U1-GPIO4)
Routing:
- net IO4: track 31.8 -> 0.00 mm, vias 1 -> 0
- net LORA_IO0: track 29.8 -> 4.00 mm
- net EN: track 30.5 -> 5.69 mm
- net IO1: track 21.6 -> 0.00 mm, vias 2 -> 1
- net GPA5: track 0.00 -> 21.6 mm, vias 0 -> 1
- net IO8: track 36.7 -> 18.3 mm
- net GPS_1PPS: track 36.1 -> 19.4 mm
- net GPS_TXD: track 26.2 -> 10.2 mm
- net Net-(U1-GPIO4): track 0.00 -> 15.4 mm, vias 0 -> 1
- net IO0: track 21.0 -> 5.71 mm
- net MISOA: track 19.8 -> 6.02 mm, vias 2 -> 1
- net SCKA: track 16.5 -> 4.31 mm, vias 2 -> 1
- net Net-(SW2A-B): track 19.2 -> 7.16 mm
- net GPS_RXD: track 20.1 -> 12.0 mm
- net SPICS0: track 14.4 -> 8.10 mm, vias 2 -> 1
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Other:
- board text removed: "RADIO ANT"

Commit message: Cleanup and update project files.
Parts:
- removed J5: Conn_01x07_Pin, Connector_PinSocket_2.54mm:PinSocket_1x07_P2.54mm_Horizontal
- removed R38: 33Ω, PCM_JLCPCB:R_0805
- added J3: Conn_01x04_Pin, Connector_PinSocket_2.54mm:PinSocket_1x04_P2.54mm_Horizontal, F.Cu at (172.5, 119.0)
- added MK1: SPH0645LM4H, Sensor_Audio:Knowles_SPH0645LM4H-6_3.5x2.65mm, F.Cu at (144.3, 121.8)
- added R43: 33Ω, PCM_JLCPCB:R_0402, F.Cu at (135.5, 122.8)
- added U12: HJ-SMA275, my_footprints:SMA-SMD_BWSMA-KE-P001, F.Cu at (185.5, 112.0)
- added U14: MAX98357A, Package_DFN_QFN:TQFN-16-1EP_3x3mm_P0.5mm_EP1.23x1.23mm, F.Cu at (139.5, 121.7)
- J1: footprint Lora-device:TF-SMD_TF-01A -> my_footprints:TF-SMD_TF-01A
- R39, R40: footprint PCM_JLCPCB:R_0805 -> PCM_JLCPCB:R_0402
- U11: footprint Lora-device:GPSM-SMD_18P-L10.1-W9.7-P1.10 -> my_footprints:GPSM-SMD_18P-L10.1-W9.7-P1.10
- U4: footprint Lora-device:USB-C-SMD_HANBO_MC-121-L119 -> my_footprints:USB-C-SMD_HANBO_MC-121-L119
- U7: footprint Lora-device:SOT-23-5_L3.0-W1.7-P0.95-LS2.8-BR -> my_footprints:SOT-23-5_L3.0-W1.7-P0.95-LS2.8-BR
- moved R39 32.5 mm to (135.5, 119.2)
- moved R40 31.9 mm to (135.5, 121.0)
- moved RESET1 21.1 mm to (164.2, 121.0), turned to -90 degrees
- moved FLASH1 19.8 mm to (168.0, 121.0), turned to -90 degrees
- moved R22 17.2 mm to (163.2, 117.4), turned to 180 degrees
- moved C15 15.8 mm to (165.2, 117.4), turned to 0 degrees
- moved R21 14.5 mm to (169.0, 117.3), turned to 0 degrees
- moved SW1 2.08 mm to (155.5, 121.9)
- moved SW3 2.08 mm to (149.3, 121.9)
Connections:
- R39 pad 1: IO4 -> IO1
- R39 pad 2: Net-(U1-GPIO4) -> Net-(U1-GPIO1)
- R40 pad 1: IO1 -> IO4
- R40 pad 2: Net-(U1-GPIO1) -> Net-(U1-GPIO4)

Commit message: Backing up.
Parts:
- removed BZ1: Buzzer, Buzzer_Beeper:MagneticBuzzer_CUI_CMT-8504-100-SMT
- removed D5: 1N4148W, Diode_SMD:D_SOD-123
- removed J1: Micro_SD_Card_Det1, my_footprints:TF-SMD_TF-01A
- removed Q2: S8050, PCM_JLCPCB:Q_SOT-23
- removed SW1, SW3: CK_KMS2xxGP, Button_Switch_SMD:SW_SPST_CK_KMS2xxGP
- removed U14: MAX98357A, Package_DFN_QFN:TQFN-16-1EP_3x3mm_P0.5mm_EP1.23x1.23mm
- removed U5: Ai-Thinker-Ra-01, RF_Module:Ai-Thinker-Ra-01-LoRa
- added C46: 100nF, PCM_JLCPCB:C_0402, F.Cu at (141.0, 107.0)
- added C47: 10uF, PCM_JLCPCB:C_0402, F.Cu at (141.0, 108.0)
- added C48: 10uF, PCM_JLCPCB:C_0402, F.Cu at (141.0, 109.0)
- added C49: 10uF, PCM_JLCPCB:C_0402, F.Cu at (130.0, 100.5)
- added JP3: SolderJumper_3_Open, Jumper:SolderJumper-3_P1.3mm_Open_RoundedPad1.0x1.5mm, F.Cu at (131.5, 108.1)
- added R38: 2.2kΩ, PCM_JLCPCB:R_0402, F.Cu at (138.0, 111.0)
- added TP1: TestPoint, TestPoint:TestPoint_THTPad_1.0x1.0mm_Drill0.5mm, F.Cu at (116.3, 98.0)
- added U15: HJ-SMA275, LoRa_library:SMA-SMD_BWSMA-KE-P001, F.Cu at (185.1, 112.1)
- added U16: Black_headphone_jack, LoRa_library:AUDIO-TH_320B, F.Cu at (155.2, 119.1)
- added U17: RA-01SH-P, LoRa_library:COMM-SMD_17P-L17.0-W16.0-P2.00_RA-01S-P, F.Cu at (169.1, 107.3)
- added U18: L76KB-A58, LoRa_library:GPSM-SMD_18P-L10.1-W9.7-P1.10, F.Cu at (158.9, 90.2)
- added U19: TF-01A, LoRa_library:TF-SMD_TF-01A, F.Cu at (172.4, 84.3)
- added U20: MAX98357AETE+T, LoRa_library:TQFN-16_L3.0-W3.0-P0.50-BL-EP1.5, F.Cu at (137.8, 107.9)
- R5: value 330Ω -> 33Ω
- U11: value L76KB-A58 -> MC-121-L119; footprint my_footprints:GPSM-SMD_18P-L10.1-W9.7-P1.10 -> LoRa_library:USB-C-SMD_HANBO_MC-121-L119
- U12: value HJ-SMA275 -> K2-1102AQ-K4CW-01; footprint my_footprints:SMA-SMD_BWSMA-KE-P001 -> LoRa_library:KEY-TH_K2-1102AQ-KXXW-XX
- U4: value MC-121-L119 -> STLQ015M33R; footprint my_footprints:USB-C-SMD_HANBO_MC-121-L119 -> LoRa_library:SOT-23-5_L3.0-W1.7-P0.95-LS2.8-BR
- U7: value STLQ015M33R -> K2-1102AQ-K4CW-01; footprint my_footprints:SOT-23-5_L3.0-W1.7-P0.95-LS2.8-BR -> LoRa_library:KEY-TH_K2-1102AQ-KXXW-XX
- moved U11 44.4 mm to (124.7, 119.5), turned to 0 degrees
- moved R5 41.0 mm to (135.5, 110.6), turned to 0 degrees
- moved R21 40.8 mm to (147.0, 83.0)
- moved C15 40.8 mm to (143.2, 83.0)
- moved FLASH1 40.8 mm to (146.0, 86.7)
- moved R22 40.8 mm to (141.2, 83.0)
- moved RESET1 40.8 mm to (142.2, 86.6)
- moved J3 37.6 mm to (134.9, 118.9)
- moved U4 34.1 mm to (149.5, 92.2), turned to -90 degrees
- moved U7 32.2 mm to (164.3, 120.4), turned to 0 degrees
- moved R4 32.2 mm to (152.4, 108.0), turned to 180 degrees
- moved R42 30.7 mm to (134.9, 116.0), turned to -90 degrees
- moved DNP4 29.4 mm to (178.6, 97.2), turned to -90 degrees
- moved R41 28.9 mm to (137.4, 116.0), turned to -90 degrees
- moved L1 26.4 mm to (176.4, 96.7), turned to 0 degrees
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Connections:
- net BUZZER renamed IO21
- C34 pad 1: Net-(U11-V_BCKP) -> Net-(U18-V_BCKP)
- DNP6 pad 1: Net-(U11-RF_IN) -> Net-(U18-RF_IN)
- MK1 pad 2: unconnected-(MK1-SEL-Pad2) -> GND
- MK1 pad 3: unconnected-(MK1-GND-Pad3) -> GND
- MK1 pad 5: unconnected-(MK1-VDD-Pad5) -> VDD_CPU
- R32 pad 1: GPA6 -> Net-(U10-ST)
- R34 pad 2: Net-(U4-CC1) -> Net-(U11-CC1)
- R35 pad 2: Net-(U4-CC2) -> Net-(U11-CC2)
- R36 pad 2: Net-(U11-VDD_RF) -> Net-(U18-VDD_RF)
- R8 pad 1: Net-(U11-SET) -> Net-(U18-SET)
- R9 pad 1: Net-(U11-RF_IN) -> Net-(U18-RF_IN)
- U10 pad 8: GPA6 -> Net-(U10-ST)
- U11 pad 13: unconnected-(U11-ANTON-Pad13) -> GND
- U12 pad 1: GND -> IO17
- U6 pad 1: Net-(U4-DN1) -> Net-(U11-DN1)
- U6 pad 3: Net-(U4-DP1) -> Net-(U11-DP1)
- U7 pad 1: VBAT -> GPB7
- U7 pad 3: VBAT -> GND
- U7 pad 4: unconnected-(U7-NC-Pad4) -> GND
Routing:
- net VBAT: track 54.9 -> 0.00 mm
- net TOUCH_IRQ: track 44.5 -> 0.00 mm, vias 2 -> 0
- net MISOB: track 44.3 -> 0.00 mm, vias 1 -> 0
- net MOSIB: track 43.1 -> 0.00 mm, vias 2 -> 0
- net IO11/BAT: track 38.9 -> 0.00 mm, vias 2 -> 0
- net +5V: track 52.3 -> 13.5 mm
- net SCKB: track 38.3 -> 0.00 mm, vias 1 -> 0
- net SCREEN_LED: track 33.1 -> 0.00 mm, vias 1 -> 0
- net SCREEN_DC: track 32.5 -> 0.00 mm, vias 2 -> 0
- net SCREEN_CS: track 29.5 -> 0.00 mm
- net TOUCH_CS: track 29.3 -> 0.00 mm, vias 2 -> 0
- net SCREEN_RST: track 24.7 -> 0.00 mm
- net (no net): track 23.7 -> 0.00 mm, vias 4 -> 0
- net GPA5: track 21.6 -> 0.00 mm, vias 1 -> 0
- net GPS_1PPS: track 19.4 -> 0.00 mm, vias 1 -> 0
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
Commit message: To be routed, most work likely done.
Parts:
- removed R1: 10K, Resistor_SMD:R_0402_1005Metric
- removed R41: 4.7kΩ, PCM_JLCPCB:R_0402
- removed SW2: SW_DPST_x2, Connector_PinHeader_2.54mm:PinHeader_1x02_P2.54mm_Vertical
- removed U13: MCP23S17_ML, Package_DFN_QFN:QFN-28-1EP_6x6mm_P0.65mm_EP4.25x4.25mm
- removed U20: MAX98357AETE+T, LoRa_library:TQFN-16_L3.0-W3.0-P0.50-BL-EP1.5
- added J1: Micro_SD_Card_Det1, my_footprints:TF-SMD_TF-01A, F.Cu at (172.5, 84.2)
- added R44: 33Ω, PCM_JLCPCB:R_0402, F.Cu at (158.8, 102.2)
- added R45: 33Ω, PCM_JLCPCB:R_0402, F.Cu at (158.8, 100.3)
- added R46: 33Ω, PCM_JLCPCB:R_0402, F.Cu at (158.8, 98.5)
- added R47: 2.2kΩ, PCM_JLCPCB:R_0402, F.Cu at (149.2, 109.8)
- added R48: 2.2kΩ, PCM_JLCPCB:R_0402, F.Cu at (148.2, 109.8)
- added U14: MCP23017_ML, Package_DFN_QFN:QFN-28-1EP_6x6mm_P0.65mm_EP4.25x4.25mm, F.Cu at (150.4, 104.8)
- added U5: SK-12D02-VG5, LoRa_library:SW-TH_SK-12D02-VG5, F.Cu at (185.8, 86.8)
- G***: moved to F.Cu
- J2: footprint Connector_PinHeader_2.54mm:PinHeader_1x02_P2.54mm_Vertical -> Connector_PinHeader_1.27mm:PinHeader_1x02_P1.27mm_Vertical
- R24: value 470R -> 330Ω; footprint Resistor_SMD:R_0402_1005Metric -> PCM_JLCPCB:R_0402
- R4: value 10K -> 10kΩ; footprint Resistor_SMD:R_0402_1005Metric -> PCM_JLCPCB:R_0402
- R42: value 4.7kΩ -> 330Ω
- U19: value TF-01A -> MAX98357A; footprint LoRa_library:TF-SMD_TF-01A -> Package_DFN_QFN:TQFN-16-1EP_3x3mm_P0.5mm_EP1.23x1.23mm
- moved U19 47.1 mm to (131.0, 106.5), turned to 0 degrees
- moved R24 25.8 mm to (155.9, 103.5)
- moved R42 22.8 mm to (155.9, 107.2), turned to 0 degrees
- moved R31 12.4 mm to (169.7, 92.0), turned to 90 degrees
- moved C48 11.5 mm to (129.6, 109.8), turned to -90 degrees
- moved R38 10.7 mm to (127.8, 107.5)
- moved C47 10.6 mm to (130.5, 109.8), turned to -90 degrees
- moved G*** 10.3 mm to (140.0, 111.4), turned to 0 degrees
- moved C46 9.90 mm to (131.5, 109.8), turned to -90 degrees
- moved R5 9.27 mm to (127.8, 105.4), turned to -90 degrees
- moved JP3 4.86 mm to (131.6, 113.0), turned to 0 degrees
- moved R39 3.77 mm to (131.5, 103.2), turned to 90 degrees
- moved C43 3.58 mm to (145.6, 108.3), turned to -90 degrees
- moved R4 1.51 mm to (153.8, 108.7)
- moved R40 1.41 mm to (130.3, 103.3), turned to 90 degrees
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Connections:
- DNP2 pad 1: Net-(U5-ANT) -> Net-(U17-ANT)
- J3 pad 1: U0TXD/IO43 -> U0TXD/IO43/I2C_SCK
- J3 pad 2: U0RXD/IO44 -> U0RXD/IO44/I2C_SDA
- J8 pad 3: (no net) -> GND
- L1 pad 1: Net-(U5-ANT) -> Net-(U17-ANT)
- R12 pad 2: IO11/BAT -> IO9/BAT
- R19 pad 1: IO11/BAT -> IO9/BAT
- R24 pad 1: Net-(U1-U0TXD) -> Net-(U1-U0RXD)
- R24 pad 2: U0TXD/IO43 -> U0RXD/IO44/I2C_SDA
- R38 pad 2: Net-(U14-~{SD_MODE}) -> Net-(U19-~{SD_MODE})
- R4 pad 2: EXP_RST -> SPICLK_P/IO47/EXP_RST
- R42 pad 1: VDD_CPU -> Net-(U1-U0TXD)
- R42 pad 2: U0TXD/IO43 -> U0TXD/IO43/I2C_SCK
- R5 pad 2: Net-(U14-DIN) -> Net-(U19-DIN)
- U1 pad 11: TOUCH_IRQ -> TOUCH_CS
- U1 pad 12: GPS_1PPS -> LORA_BUSY
- U1 pad 14: SCREEN_LED -> IO9/BAT
- U1 pad 16: IO11/BAT -> SCREEN_LED
- U1 pad 23: IO17 -> SD_CS
- U1 pad 37: SPICLK_P/IO47/EXP_CS -> SPICLK_P/IO47/EXP_RST
- U1 pad 50: U0RXD/IO44 -> Net-(U1-U0RXD)
- U1 pad 7: LORA_IO0 -> SCREEN_CS
- U12 pad 1: IO17 -> GPA7
- U16 pad 3: Net-(U14-OUTN) -> Net-(U16-GND)
- U16 pad 4: Net-(U14-OUTP) -> Net-(U16-L)
- U17 pad 1: unconnected-(U17-ANT-Pad1) -> Net-(U17-ANT)
- U17 pad 10: unconnected-(U17-BUSY-Pad10) -> LORA_BUSY
- U17 pad 11: unconnected-(U17-RF_EN-Pad11) -> LORA_RF_EN
- U17 pad 12: unconnected-(U17-SCK-Pad12) -> SCKA
- U17 pad 13: unconnected-(U17-MISO-Pad13) -> MISOA
- U17 pad 14: unconnected-(U17-MOSI-Pad14) -> MOSIA
- U17 pad 15: unconnected-(U17-NSS-Pad15) -> SPICLK_N/IO48/LORA_CS
- U17 pad 16: unconnected-(U17-GND-Pad16) -> GND
- U17 pad 17: unconnected-(U17-GND-Pad17) -> GND
- U17 pad 2: unconnected-(U17-GND-Pad2) -> GND
- U17 pad 3: unconnected-(U17-3V3-Pad3) -> VDD_CPU
- U17 pad 4: unconnected-(U17-RESET-Pad4) -> LORA_RST
- U17 pad 6: unconnected-(U17-DIO1-Pad6) -> Net-(U17-DIO1)
- U17 pad 7: unconnected-(U17-DIO2-Pad7) -> Net-(U17-DIO2)
- U17 pad 8: unconnected-(U17-DIO3-Pad8) -> Net-(U17-DIO3)
- U17 pad 9: unconnected-(U17-GND-Pad9) -> GND
- U19 pad 1: unconnected-(U19-DAT2(RSV)-Pad1) -> Net-(U19-DIN)
- U19 pad 10: unconnected-(U19-GND-Pad10) -> Net-(U16-GND)
- U19 pad 11: unconnected-(U19-GND-Pad11) -> GND
- U19 pad 2: unconnected-(U19-CDDAT3(CS)-Pad2) -> Net-(JP3-C)
- U19 pad 3: unconnected-(U19-CMD(DI)-Pad3) -> GND
- U19 pad 4: unconnected-(U19-VDD-Pad4) -> Net-(U19-~{SD_MODE})
- U19 pad 7: unconnected-(U19-DAT0(D0)-Pad7) -> VDD_CPU
- U19 pad 8: unconnected-(U19-DAT1(RSV)-Pad8) -> VDD_CPU
- U19 pad 9: unconnected-(U19-CD-Pad9) -> Net-(U16-L)
Other:
- board text added: "+-"
- board text removed: "+ -"

Commit message: new case design.
Parts:
- moved R14 5.81 mm to (176.8, 91.5)
- moved R32 5.00 mm to (117.2, 96.8), turned to -90 degrees
- moved R10 4.62 mm to (174.2, 116.0), turned to 180 degrees
- moved C13 4.59 mm to (132.9, 100.8)
- moved C32 4.59 mm to (134.1, 100.8)
- moved R13 4.20 mm to (107.2, 87.3), turned to 180 degrees
- moved C30 3.95 mm to (173.6, 91.5), turned to -90 degrees
- moved R27 3.41 mm to (129.5, 96.0), turned to 0 degrees
- moved R37 3.00 mm to (177.9, 91.5)
- moved R26 2.90 mm to (129.5, 94.9), turned to 0 degrees
- moved R17 2.81 mm to (170.2, 91.5)
- moved C49 1.92 mm to (131.9, 100.8), turned to -90 degrees
- moved R31 1.88 mm to (171.4, 91.5)
- moved C36 1.54 mm to (172.3, 96.0), turned to 90 degrees
- moved TP1 1.42 mm to (115.5, 96.8)
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Connections:
- net U0RXD/IO44/I2C_SDA renamed MTMS/IO42/I2C_SDA
- net U0TXD/IO43/I2C_SCK renamed MTDO/IO40/I2C_SCK
- R24 pad 1: Net-(U1-U0RXD) -> Net-(U1-MTMS)
- R42 pad 1: Net-(U1-U0TXD) -> Net-(U1-MTDO)
- U1 pad 45: GPS_RXD -> Net-(U1-MTDO)
- U1 pad 48: GPS_TXD -> Net-(U1-MTMS)
- U1 pad 49: Net-(U1-U0TXD) -> GPS_RXD
- U1 pad 50: Net-(U1-U0RXD) -> GPS_TXD
Routing:
- net VBAT: track 0.00 -> 95.9 mm, vias 0 -> 3
- net MOSIA: track 0.00 -> 86.5 mm, vias 0 -> 4
- net SCKA: track 0.00 -> 81.7 mm, vias 0 -> 4
- net MISOA: track 0.00 -> 71.7 mm, vias 0 -> 4
- net LORA_BUSY: track 0.00 -> 69.9 mm, vias 0 -> 4
- net SCREEN_RST: track 0.00 -> 68.6 mm, vias 0 -> 4
- net SPICLK_N/IO48/LORA_CS: track 0.00 -> 67.6 mm, vias 0 -> 2
- net Net-(U8-~{ON}): track 0.00 -> 67.5 mm, vias 0 -> 4
- net IO10: track 0.00 -> 58.7 mm, vias 0 -> 4
- net GPA5: track 0.00 -> 53.1 mm, vias 0 -> 4
- net GPA6: track 0.00 -> 52.7 mm, vias 0 -> 2
- net TOUCH_IRQ: track 0.00 -> 52.2 mm, vias 0 -> 2
- net MISOB: track 0.00 -> 46.9 mm, vias 0 -> 2
- net GPB6: track 0.00 -> 45.1 mm, vias 0 -> 2
- net Net-(U1-MTDO): track 0.00 -> 44.9 mm, vias 0 -> 2
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