File: LoRa-device.kicad_sch (KiCad schematic)
At the start: 121 parts, among them J1 Connector, USB-TYPE-C-16P, J2 Conn_01x02_Pin, J3 Conn_Coaxial, J4 Conn_01x14_Pin, J6 Conn_01x04_Pin, J7 Screw_Terminal_01x08, J8 U.FL, Q2 S8050, SW2 SW_DPST_x2, U1 ESP32-S3, U10 TPS2116DRL, U11 L76KB-A58, U13 MCP23S17_ML, U2 W25Q128JVS, U3 TP4055, U5 Ai-Thinker-Ra-01, U6 USBLC6-2P6, U7 STLQ015M33R, U8 TPS22917LDBV, U9 AP63203WU, Y1 32.768 kHz, Y2 40MHz(10ppm)

Commit message: Major overhaul of version A
Parts:
- removed C30: 1uF, PCM_JLCPCB:C_0402, symbol PCM_JLCPCB-Capacitors:0402,1uF
- removed J1: Connector, USB-TYPE-C-16P, PCM_JLCPCB:TYPE-C-SMD_HX-TYPE-C-16PIN, symbol PCM_JLCPCB-Extended:Connector, USB-TYPE-C-16P
- removed J7: Screw_Terminal_01x08, Connector_Phoenix_MC:PhoenixContact_MC_1,5_8-G-3.81_1x08_P3.81mm_Horizontal, symbol Connector:Screw_Terminal_01x08
- removed R14, R17: 5.1K, Resistor_SMD:R_0402_1005Metric, symbol Device:R
- removed R40: 100kΩ, PCM_JLCPCB:R_0402, symbol PCM_JLCPCB-Resistors:0402,100kΩ
- removed R41: 47Ω, PCM_JLCPCB:R_0402, symbol PCM_JLCPCB-Resistors:0402,47Ω
- removed TP2: TestPoint_2Pole, TestPoint:TestPoint_2Pads_Pitch2.54mm_Drill0.8mm, symbol Connector:TestPoint_2Pole
- added J1: Micro_SD_Card_Det1, Lora-device:TF-SMD_TF-01A, symbol Connector:Micro_SD_Card_Det1
- added MK1: SPH0645LM4H, Sensor_Audio:Knowles_SPH0645LM4H-6_3.5x2.65mm, symbol Sensor_Audio:SPH0645LM4H
- added R34, R35: 5.1K, Resistor_SMD:R_0402_1005Metric, symbol Device:R
- added U4: MC-121-L119, Lora-device:USB-C-SMD_HANBO_MC-121-L119, symbol Lora-device:MC-121-L119
- J3: footprint Connector_Coaxial:SMA_Molex_73251-1153_EdgeMount_Horizontal -> Lora-device:SMA-SMD_BWSMA-KE-P001
Connections:
- net +5V: now also U4.A4B9 (VBUS), U4.B4A9 (VBUS)
- net GND: now also R34.1, R35.1, U4.13 (EH), U4.A1B12 (GND), U4.B1A12 (GND)
- net MOSIA: no longer J6.2 (Pin_2)
- net SCKA: no longer J6.4 (Pin_4)
- net SCREEN_CS: now also U13.1 (GPB4); no longer U1.15 (GPIO10)
- net SD_CS: now also U13.24 (GPA7); no longer J6.1 (Pin_1), U1.12 (GPIO7)
- net TOUCH_CS: now also U13.2 (GPB5); no longer U1.24 (GPIO18)
- net LORA_IO4: now reaches U5.10 (DIO4)
- net LORA_IO4: now also U13.27 (GPB2)
- net LORA_IO5: now reaches U5.11 (DIO5)
- net LORA_IO5: now also U13.28 (GPB3)
- net GPS_1PPS: now reaches U11.4 (1PPS)
- net GPS_1PPS: now also U1.12 (GPIO7)
- net LORA_IO2: now reaches U5.7 (DIO2)
- net LORA_IO2: now also U13.25 (GPB0)
- net LORA_IO3: now reaches U5.8 (DIO3)
- net LORA_IO3: now also U13.26 (GPB1)
- net at U6.1 (I/O1): now also U4.A7 (DN1), U4.B7 (DN2)
- net at U6.3 (I/O2): now also U4.A6 (DP1), U4.B6 (DP2)
- net IO18: now reaches U13.15 (INTB)
- net IO18: now also U1.24 (GPIO18)
- net IO10: now reaches U13.16 (INTA)
- net IO10: now also U1.15 (GPIO10)
- net GPB6: now reaches U13.3 (GPB6)
- net GPB7: now reaches U13.4 (GPB7)
- new net: R34.2, U4.A5 (CC1)
- new net: R35.2, U4.B5 (CC2)
- no-connect marks 22 -> 17
Other:
- note added: "HEADER"
- note added: "I2S MICROPHONE"
- note added: "ILI9341"
- note added: "MICRO SD CARD"
- note removed: "HEADER PINS"
- note removed: "ILI9341/SD CARD"
- moved on the sheet: BZ1, C13, C16, C17, C3, C32, C36, C39, C40, C6, C7, D2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

Commit message: Just a backup.
Parts:
- removed MK1: SPH0645LM4H, Sensor_Audio:Knowles_SPH0645LM4H-6_3.5x2.65mm, symbol Sensor_Audio:SPH0645LM4H
- added C30: 100nF, PCM_JLCPCB:C_0402, symbol PCM_JLCPCB-Capacitors:0402,100nF
- added C44: 220pF, PCM_JLCPCB:C_0402, symbol PCM_JLCPCB-Capacitors:0402,220pF
- added C45: 1uF, PCM_JLCPCB:C_0402, symbol PCM_JLCPCB-Capacitors:0402,1uF
- added J5: Conn_01x07_Pin, Connector_PinSocket_2.54mm:PinSocket_1x07_P2.54mm_Horizontal, symbol Connector:Conn_01x07_Pin
- added R14, R17, R37: 10K, Resistor_SMD:R_0402_1005Metric, symbol Device:R
- added R38, R39, R40: 33Ω, PCM_JLCPCB:R_0805, symbol PCM_JLCPCB-Resistors:0805,33Ω
- added R41, R42: 4.7kΩ, PCM_JLCPCB:R_0402, symbol PCM_JLCPCB-Resistors:0402,4.7kΩ
- added SW1, SW3: CK_KMS2xxGP, Button_Switch_SMD:SW_SPST_CK_KMS2xxGP, symbol Switch:CK_KMS2xxGP
Connections:
- net +3V3: now also J1.4 (VDD), C30.1, C44.1, C45.1, J5.7 (Pin_7), R14.1, R17.1, R37.1, R41.1, R42.1
- net GND: now also J1.10 (SHIELD), J1.6 (VSS), C30.2, C44.2, C45.2, J5.6 (Pin_6), SW1.1, SW1.SH (B), SW3.1, SW3.SH (B)
- net GPB6: now also J1.9 (DET)
- net GPB7: now also SW1.2
- net IO1: now also J5.3 (Pin_3), R40.1; no longer U1.6 (GPIO1)
- net IO17: now also SW3.2
- net IO4: now also J5.4 (Pin_4), R39.1; no longer U1.9 (GPIO4)
- net IO8: now also R38.2
- net MISOA: now also J1.7 (DAT0), R14.2
- net MOSIA: now also J1.3 (CMD)
- net SCKA: now also J1.5 (CLK)
- net SD_CS: now also J1.2 (DAT3/CD)
- net U0RXD/IO44: now also J5.2 (Pin_2), R41.2
- net U0TXD/IO43: now also J5.1 (Pin_1), R42.2
- net at J1.1 (DAT2): now also R17.2
- net at J1.8 (DAT1): now also R37.2
- new net: R40.2, U1.6 (GPIO1)
- new net: R39.2, U1.9 (GPIO4)
- new net: J5.5 (Pin_5), R38.1
- no-connect marks 17 -> 21
Other:
- note added: "BUTTONS"
- note added: "I2S/I2C HEADER"
- note removed: "I2S MICROPHONE"
- moved on the sheet: C33, J1, J6

Commit message: Cleanup and update project files.
Parts:
- removed J3: Conn_Coaxial, Lora-device:SMA-SMD_BWSMA-KE-P001, symbol Connector:Conn_Coaxial
- removed J5: Conn_01x07_Pin, Connector_PinSocket_2.54mm:PinSocket_1x07_P2.54mm_Horizontal, symbol Connector:Conn_01x07_Pin
- removed R38, R39, R40: 33Ω, PCM_JLCPCB:R_0805, symbol PCM_JLCPCB-Resistors:0805,33Ω
- added J3: Conn_01x04_Pin, Connector_PinSocket_2.54mm:PinSocket_1x04_P2.54mm_Horizontal, symbol Connector:Conn_01x04_Pin
- added MK1: SPH0645LM4H, Sensor_Audio:Knowles_SPH0645LM4H-6_3.5x2.65mm, symbol Sensor_Audio:SPH0645LM4H
- added R39, R40, R43: 33Ω, PCM_JLCPCB:R_0402, symbol PCM_JLCPCB-Resistors:0402,33Ω
- added U12: HJ-SMA275, my_footprints:SMA-SMD_BWSMA-KE-P001, symbol SMA_connector:HJ-SMA275
- added U14: MAX98357A, Package_DFN_QFN:TQFN-16-1EP_3x3mm_P0.5mm_EP1.23x1.23mm, symbol Audio:MAX98357A
- J1: footprint Lora-device:TF-SMD_TF-01A -> my_footprints:TF-SMD_TF-01A
- SW1, SW3: LCSC (none) -> C221698
- U11: footprint Lora-device:GPSM-SMD_18P-L10.1-W9.7-P1.10 -> my_footprints:GPSM-SMD_18P-L10.1-W9.7-P1.10
- U4: footprint Lora-device:USB-C-SMD_HANBO_MC-121-L119 -> my_footprints:USB-C-SMD_HANBO_MC-121-L119
- U7: footprint Lora-device:SOT-23-5_L3.0-W1.7-P0.95-LS2.8-BR -> my_footprints:SOT-23-5_L3.0-W1.7-P0.95-LS2.8-BR
Connections:
- net +3V3: now also J3.4 (Pin_4), MK1.5 (VDD)
- net GND: now also J3.3 (Pin_3), MK1.2 (SEL), MK1.3 (GND), U12.1, U12.2, U12.3, U12.4
- net IO1: now also MK1.1 (WS), R39.1
- net IO4: now also MK1.4 (BCLK), R40.1
- net IO8: now also R43.2
- net U0RXD/IO44: now also J3.2 (Pin_2)
- net U0TXD/IO43: now also J3.1 (Pin_1)
- net at U1.6 (GPIO1): now also R39.2
- net at U1.9 (GPIO4): now also R40.2
- net at DNP4.1, L1.2: now also U12.5
- new net: MK1.6 (DATA), R43.1
- new net: U14.11 (GND), U14.15 (GND), U14.3 (GND)
- new net: U14.7 (VDD), U14.8 (VDD)
Other:
- note added: "I2C HEADER"
- note removed: "I2S/I2C HEADER"
- moved on the sheet: C44, C45, L1, R10, R41, R42

Commit message: Backing up.
Parts:
- removed BZ1: Buzzer, Buzzer_Beeper:MagneticBuzzer_CUI_CMT-8504-100-SMT, symbol Device:Buzzer
- removed D5: 1N4148W, Diode_SMD:D_SOD-123, symbol Diode:1N4148W
- removed Q2: S8050, PCM_JLCPCB:Q_SOT-23, symbol PCM_JLCPCB-Transistors:NPN,S8050
- removed R5: 330Ω, PCM_JLCPCB:R_0402, symbol PCM_JLCPCB-Resistors:0402,330Ω
- removed SW1, SW3: CK_KMS2xxGP, Button_Switch_SMD:SW_SPST_CK_KMS2xxGP, symbol Switch:CK_KMS2xxGP
- removed U11: L76KB-A58, my_footprints:GPSM-SMD_18P-L10.1-W9.7-P1.10, symbol Lora-device:L76KB-A58
- removed U12: HJ-SMA275, my_footprints:SMA-SMD_BWSMA-KE-P001, symbol SMA_connector:HJ-SMA275
- removed U4: MC-121-L119, my_footprints:USB-C-SMD_HANBO_MC-121-L119, symbol Lora-device:MC-121-L119
- removed U7: STLQ015M33R, my_footprints:SOT-23-5_L3.0-W1.7-P0.95-LS2.8-BR, symbol Lora-device:STLQ015M33R
- added C46: 100nF, PCM_JLCPCB:C_0402, symbol PCM_JLCPCB-Capacitors:0402,100nF
- added C47, C48, C49: 10uF, PCM_JLCPCB:C_0402, symbol PCM_JLCPCB-Capacitors:0402,10uF
- added JP3: SolderJumper_3_Open, Jumper:SolderJumper-3_P1.3mm_Open_RoundedPad1.0x1.5mm, symbol Jumper:SolderJumper_3_Open
- added R38: 2.2kΩ, PCM_JLCPCB:R_0402, symbol PCM_JLCPCB-Resistors:0402,2.2kΩ
- added R5: 33Ω, PCM_JLCPCB:R_0402, symbol PCM_JLCPCB-Resistors:0402,33Ω
- added TP1: TestPoint, TestPoint:TestPoint_THTPad_1.0x1.0mm_Drill0.5mm, symbol Connector:TestPoint
- added U11: MC-121-L119, LoRa_library:USB-C-SMD_HANBO_MC-121-L119, symbol LoRa_library:MC-121-L119
- added U12, U7: K2-1102AQ-K4CW-01, LoRa_library:KEY-TH_K2-1102AQ-KXXW-XX, symbol LoRa_library:K2-1102AQ-K4CW-01
- added U15: HJ-SMA275, LoRa_library:SMA-SMD_BWSMA-KE-P001, symbol LoRa_library:HJ-SMA275
- added U16: Black_headphone_jack, LoRa_library:AUDIO-TH_320B, symbol LoRa_library:Black_headphone_jack
- added U17: RA-01SH-P, LoRa_library:COMM-SMD_17P-L17.0-W16.0-P2.00_RA-01S-P, symbol LoRa_library:RA-01SH-P
- added U18: L76KB-A58, LoRa_library:GPSM-SMD_18P-L10.1-W9.7-P1.10, symbol LoRa_library:L76KB-A58
- added U19: TF-01A, LoRa_library:TF-SMD_TF-01A, symbol LoRa_library:TF-01A
- added U20: MAX98357AETE+T, LoRa_library:TQFN-16_L3.0-W3.0-P0.50-BL-EP1.5, symbol LoRa_library:MAX98357AETE+T
- added U4: STLQ015M33R, LoRa_library:SOT-23-5_L3.0-W1.7-P0.95-LS2.8-BR, symbol LoRa_library:STLQ015M33R
- U14: LCSC (none) -> C910544
Connections:
- net +3V3: now also U14.7 (VDD), U14.8 (VDD), C46.1, C47.1, C48.1, JP3.3 (B), U18.8 (VCC)
- net +5V: now also U11.A4B9 (VBUS), U11.B4A9 (VBUS)
- net GND: now also U14.11 (GND), U14.15 (GND), U14.17 (PAD), U14.3 (GND), C46.2, C47.2, C48.2, C49.2, JP3.1 (A), U11.13 (EH), U11.A1B12 (GND), U11.B1A12 (GND), U12.2, U12.3, U12.4, U15.1, U15.2, U15.3, U15.4, U18.1 (GND), U18.10 (GND), U18.12 (GND), U4.2 (GND), U7.2, U7.3, U7.4
- net GPA6: now also R38.1; no longer R32.1, U10.8 (ST)
- net GPB7: now also U7.1
- net GPS_1PPS: now also U18.4 (1PPS)
- net GPS_RST: now also U18.9 (RESET_N)
- net GPS_RXD: now also U18.3 (RXD)
- net GPS_TXD: now also U18.2 (TXD)
- net GPS_WKUP: now also U18.5 (WAKE_UP)
- net IO1: now also U14.14 (LRCLK)
- net IO17: now also U12.1
- net IO4: now also U14.16 (BCLK)
- net VBAT: now also U4.1 (IN), U4.3 (EN)
- net VDD_SPI: now also C49.1
- net at DNP6.1, R9.1: now also U18.11 (RF_IN)
- net at R36.2: now also U18.14 (VDD_RF)
- net at R8.1: now also U18.18 (SET)
- net at C34.1: now also U18.6 (V_BCKP), U4.5 (OUT)
- net at DNP4.1, L1.2: now also U15.5
- net at R34.2: now also U11.A5 (CC1)
- net at U6.3 (I/O2): now also U11.A6 (DP1), U11.B6 (DP2)
- net at U6.1 (I/O1): now also U11.A7 (DN1), U11.B7 (DN2)
- net at R35.2: now also U11.B5 (CC2)
- net at U14.1 (DIN): now also R5.2
- net at U14.10 (OUTN): now also U16.3 (GND)
- net at U14.2 (GAIN_SLOT): now also JP3.2 (C)
- net at U14.4 (~{SD_MODE}): now also R38.2
- net at U14.9 (OUTP): now also U16.4 (L)
- net BUZZER renamed IO21
- net IO21: now also R5.1
- new net: R32.1, TP1.1, U10.8 (ST)
- no-connect marks 21 -> 22
Other:
- note added: "12dB gain GND"
- note added: "6dB gain VDD"
- note added: "9dB gain unconnected"
- note added: "AUDIO"
- note removed: "BUZZER"
- moved on the sheet: AE1, C10, C11, C13, C14, C15, C18, C19, C25, C26, C31, C32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

Commit message: To be routed, most work likely done.
Parts:
- removed R1, R4: 10K, Resistor_SMD:R_0402_1005Metric, symbol Device:R
- removed R24: 470R, Resistor_SMD:R_0402_1005Metric, symbol Device:R
- removed R41, R42: 4.7kΩ, PCM_JLCPCB:R_0402, symbol PCM_JLCPCB-Resistors:0402,4.7kΩ
- removed SW2: SW_DPST_x2, Connector_PinHeader_2.54mm:PinHeader_1x02_P2.54mm_Vertical, symbol Switch:SW_DPST_x2
- removed U13: MCP23S17_ML, Package_DFN_QFN:QFN-28-1EP_6x6mm_P0.65mm_EP4.25x4.25mm, symbol Interface_Expansion:MCP23S17_ML
- removed U14: MAX98357A, Package_DFN_QFN:TQFN-16-1EP_3x3mm_P0.5mm_EP1.23x1.23mm, symbol Audio:MAX98357A
- removed U19: TF-01A, LoRa_library:TF-SMD_TF-01A, symbol LoRa_library:TF-01A
- removed U20: MAX98357AETE+T, LoRa_library:TQFN-16_L3.0-W3.0-P0.50-BL-EP1.5, symbol LoRa_library:MAX98357AETE+T
- removed U5: Ai-Thinker-Ra-01, RF_Module:Ai-Thinker-Ra-01-LoRa, symbol RF_Module:Ai-Thinker-Ra-01
- added R24, R42: 330Ω, PCM_JLCPCB:R_0402, symbol PCM_JLCPCB-Resistors:0402,330Ω
- added R4: 10kΩ, PCM_JLCPCB:R_0402, symbol PCM_JLCPCB-Resistors:0402,10kΩ
- added R44, R45, R46: 33Ω, PCM_JLCPCB:R_0402, symbol PCM_JLCPCB-Resistors:0402,33Ω
- added R47, R48: 2.2kΩ, PCM_JLCPCB:R_0402, symbol PCM_JLCPCB-Resistors:0402,2.2kΩ
- added U14: MCP23017_ML, Package_DFN_QFN:QFN-28-1EP_6x6mm_P0.65mm_EP4.25x4.25mm, symbol Interface_Expansion:MCP23017_ML
- added U19: MAX98357A, Package_DFN_QFN:TQFN-16-1EP_3x3mm_P0.5mm_EP1.23x1.23mm, symbol Audio:MAX98357A
- added U5: SK-12D02-VG5, LoRa_library:SW-TH_SK-12D02-VG5, symbol LoRa_library:SK-12D02-VG5
- J2: footprint Connector_PinHeader_2.54mm:PinHeader_1x02_P2.54mm_Vertical -> Connector_PinHeader_1.27mm:PinHeader_1x02_P1.27mm_Vertical
Connections:
- net LORA_IO0 is gone; now on net SCREEN_CS: U1.7 (GPIO2)
- net +3V3: now also U17.3 (3V3), R4.1, R47.1, R48.1, U14.5 (VDD), U19.7 (VDD), U19.8 (VDD)
- net GND: now also J1.11 (SHIELD), J1.12 (SHIELD), J1.13 (SHIELD), J8.3 (Ext), U17.16 (GND), U17.17 (GND), U17.2 (GND), U17.9 (GND), U14.11 (A0), U14.12 (A1), U14.13 (A2), U14.29 (EP), U14.6 (VSS), U19.11 (GND), U19.15 (GND), U19.17 (PAD), U19.3 (GND), U5.2, U5.4, U5.5
- net GPA5: now also U14.22 (GPA5)
- net GPA6: now also U14.23 (GPA6)
- net GPB6: now also U14.3 (GPB6)
- net GPB7: now also U14.4 (GPB7)
- net GPS_1PPS: now also U14.28 (GPB3); no longer U1.12 (GPIO7)
- net GPS_RST: now also U14.20 (GPA3)
- net GPS_WKUP: now also U14.21 (GPA4)
- net IO1: now also U19.14 (LRCLK)
- net IO10: now also U14.16 (INTA)
- net IO18: now also U14.15 (INTB)
- net IO4: now also U19.16 (BCLK)
- net LORA_IO1: now also R44.1, U14.18 (GPA1)
- net LORA_IO2: now also R45.1, U14.25 (GPB0)
- net LORA_IO3: now also R46.1, U14.26 (GPB1)
- net LORA_RST: now also U17.4 (RESET), U14.17 (GPA0)
- net MISOA: now also U17.13 (MISO)
- net MOSIA: now also U17.14 (MOSI)
- net SCKA: now also U17.12 (SCK)
- net SCREEN_LED: now also U1.16 (GPIO11); no longer U1.14 (GPIO9)
- net SCREEN_RST: now also U14.19 (GPA2)
- net SD_CS: now also U1.23 (GPIO17)
- net SPICLK_N/IO48/LORA_CS: now also U17.15 (NSS)
- net TOUCH_CS: now also U1.11 (GPIO6)
- net TOUCH_IRQ: now also U14.1 (GPB4); no longer U1.11 (GPIO6)
- net at U1.49 (U0TXD): now also R42.1
- net at R7.1, U8.3 (~{ON}): now also U5.3
- net at R38.2: now also U19.4 (~{SD_MODE})
- net at DNP2.1, L1.1: now also U17.1 (ANT)
- net at R5.2: now also U19.1 (DIN)
- net LORA_BUSY: now reaches U17.10 (BUSY)
- net LORA_BUSY: now also U1.12 (GPIO7)
- net LORA_RF_EN: now reaches U17.11 (RF_EN)
- net LORA_RF_EN: now also U14.27 (GPB2)
- net at U17.6 (DIO1): now also R44.2
- net at U17.7 (DIO2): now also R45.2
- net at U17.8 (DIO3): now also R46.2
- net at U16.3 (GND): now also U19.10 (OUTN)
- net at JP3.2 (C): now also U19.2 (GAIN_SLOT)
- net at U16.4 (L): now also U19.9 (OUTP)
- net IO11/BAT renamed IO9/BAT
- net IO9/BAT: now also U1.14 (GPIO9); no longer U1.16 (GPIO11)
- net IO17 renamed GPA7
- net GPA7: now also U14.24 (GPA7); no longer U1.23 (GPIO17)
- net SPICLK_P/IO47/EXP_CS renamed SPICLK_P/IO47/EXP_RST
- net SPICLK_P/IO47/EXP_RST: now also R4.2, U14.14 (~{RESET})
- net U0RXD/IO44: no longer names the net of U1.50 (U0RXD)
- net U0RXD/IO44: now also R24.1; no longer J3.2 (Pin_2)
- net U0TXD/IO43 renamed U0TXD/IO43/I2C_SCK
- net U0TXD/IO43/I2C_SCK: now also R42.2, R48.2, U14.8 (SCK)
- new net U0RXD/IO44/I2C_SDA: J3.2 (Pin_2), R24.2, R47.2, U14.9 (SDA)
- no-connect marks 22 -> 25
Other:
- moved on the sheet: C36, C44, C45, C7, DNP2, DNP4, J3, L1, R10, R22, U15

Commit message: new case design.
Connections:
- net GPS_RXD: now also U1.49 (U0TXD); no longer U1.45 (MTDO)
- net GPS_TXD: now also U1.50 (U0RXD); no longer U1.48 (MTMS)
- net at R24.1: now also U1.48 (MTMS); no longer U1.50 (U0RXD)
- net at R42.1: now also U1.45 (MTDO); no longer U1.49 (U0TXD)
- net U0RXD/IO44/I2C_SDA renamed MTMS/IO42/I2C_SDA
- net U0TXD/IO43/I2C_SCK renamed MTDO/IO40/I2C_SCK
Other:
- moved on the sheet: R24, R42

Commit message: progress
Parts:
- removed C42: 10uF, Capacitor_SMD:C_0402_1005Metric, symbol Device:C
- removed J2: Conn_01x02_Pin, Connector_PinHeader_1.27mm:PinHeader_1x02_P1.27mm_Vertical, symbol Connector:Conn_01x02_Pin
- removed U12, U7: K2-1102AQ-K4CW-01, LoRa_library:KEY-TH_K2-1102AQ-KXXW-XX, symbol LoRa_library:K2-1102AQ-K4CW-01
- added C50: 22uF, PCM_JLCPCB:C_0603, symbol PCM_JLCPCB-Capacitors:0603,22uF
- added P1: 1_25T-1-2A, LoRa_library:CONN-TH_1.25T-1-2A, symbol LoRa_library:1_25T-1-2A
- added SW1, SW2: EVQPUC02K, LoRa_library:SW-SMD_EVQPUD02K, symbol LoRa_library:EVQPUC02K
Connections:
- net GND: now also C50.2, P1.2, SW1.2, SW1.4, SW2.2, SW2.4
- net GPA7: now also SW1.3
- net GPB7: now also SW2.3
- net LORA_IO1: now also U1.24 (GPIO18); no longer U14.18 (GPA1)
- net VBAT: now also P1.1
- net VSYS: now also C50.1
- net IO18: no longer names the net of U14.15 (INTB)
- net IO18: no longer U1.24 (GPIO18)
- no-connect marks 25 -> 29

Commit message: Changed problematic components, updated case
Parts:
- added C42, C53: 1uF, PCM_JLCPCB:C_0402, symbol PCM_JLCPCB-Capacitors:0402,1uF
- added C51: 2.2uF, PCM_JLCPCB:C_0402, symbol PCM_JLCPCB-Capacitors:0402,2.2uF
- added C52: 10uF, PCM_JLCPCB:C_0402, symbol PCM_JLCPCB-Capacitors:0402,10uF
- added R1: 100kΩ, PCM_JLCPCB:R_0402, symbol PCM_JLCPCB-Resistors:0402,100kΩ
- added R41, R49, R52, R53: 10kΩ, PCM_JLCPCB:R_0402, symbol PCM_JLCPCB-Resistors:0402,10kΩ
- added R50: 330Ω, PCM_JLCPCB:R_0402, symbol PCM_JLCPCB-Resistors:0402,330Ω
- added R51: 13kΩ, PCM_JLCPCB:R_0603, symbol PCM_JLCPCB-Resistors:0603,13kΩ
- added U12: MLT-5020, LoRa_library:BUZ-SMD_L5.0-W5.5-P4.60, symbol LoRa_library:MLT-5020
- added U13: ES8311, LoRa_library:WQFN-20_L3.0-W3.0-P0.40-BL-EP1.7, symbol LoRa_library:ES8311
- added U7: BQ25185DLHR, LoRa_library:WSON-10_L2.2-W2.0-P0.40-BL-EP_TI_DLH0010A, symbol LoRa_library:BQ25185DLHR
- J3: footprint Connector_PinSocket_2.54mm:PinSocket_1x04_P2.54mm_Horizontal -> Connector_PinSocket_2.54mm:PinSocket_1x04_P2.54mm_Vertical
Connections:
- net +3V3: now also R52.1, R53.1
- net +5V: now also C42.1, C51.1, U7.10 (IN)
- net GND: now also C42.2, C51.2, C52.2, C53.2, R1.2, R41.2, R49.2, R50.2, R51.2, U7.11 (EP), U7.5 (GND)
- net VBAT: now also C53.1, U7.2 (BAT)
- net VSYS: now also C52.1, U7.1 (SYS)
- net at MK1.6 (DATA), R43.1: now also R1.1
- new net: R51.1, U7.7 (ILIM/VSET)
- new net: R53.2, U7.9 (STAT1)
- new net: R41.1, U7.4 (CE#)
- new net: R50.1, U7.8 (ISET)
- new net: R52.2, U7.3 (STAT2)
- new net: R49.1, U7.6 (TS/MR)
Other:
- moved on the sheet: MK1, R43
