File: LoRa-device.kicad_sch (KiCad schematic)
At the start: 149 parts, among them J1 Micro_SD_Card_Det1, J3 Conn_01x04_Pin, J4 Conn_01x14_Pin, J6 Conn_01x04_Pin, J8 U.FL, P1 1_25T-1-2A, P2 1_25T-1-2A, SW1 EVQPUC02K, SW2 EVQPUC02K, U1 ESP32-S3, U11 MC-121-L119, U12 TLV62569DBV, U14 MCP23017_ML, U15 HJ-SMA275, U17 RA-01SH-P, U18 L76KB-A58, U19 MAX98357A, U2 W25Q128JVS, U3 ICS-43432, U4 STLQ015M33R, U5 SK-12D02-VG5, U6 USBLC6-2P6, U7 BQ25185DLHR, U8 TPS22917LDBV, U9 MHCI04020-2R2M-R8, Y1 32.768 kHz, Y2 40MHz(10ppm)

Commit message: Production ready prototype
Parts:
- removed C10, C11, C15, C18, C19, C22, C32, C43: 0.1uF, Capacitor_SMD:C_0402_1005Metric, symbol Device:C
- removed C13, C26, C39: 1uF, Capacitor_SMD:C_0402_1005Metric, symbol Device:C
- removed C16, C25, C3, C6, C8: 10uF, Capacitor_SMD:C_0402_1005Metric, symbol Device:C
- removed C33, C37, C38, C4: 12pF, Capacitor_SMD:C_0402_1005Metric, symbol Device:C
- removed C40: 10nF, Capacitor_SMD:C_0402_1005Metric, symbol Device:C
- removed C5: 4.7uF, PCM_JLCPCB:C_0402, symbol PCM_JLCPCB-Capacitors:0402,4.7uF
- removed C9: 100nF, PCM_JLCPCB:C_0402, symbol PCM_JLCPCB-Capacitors:0402,100nF
- removed L1, R23, R24, R26, R27, R28, R29, R3, R30, R36, R9: 0R, Resistor_SMD:R_0402_1005Metric, symbol Device:R
- removed R10, R11, R13, R14, R17, R21, R22, R31, R37: 10K, Resistor_SMD:R_0402_1005Metric, symbol Device:R
- removed R12, R19: 200K, Resistor_SMD:R_0402_1005Metric, symbol Device:R
- removed R16, R25: 470R, Resistor_SMD:R_0402_1005Metric, symbol Device:R
- removed R18, R2: 33R, Resistor_SMD:R_0402_1005Metric, symbol Device:R
- removed R34, R35: 5.1K, Resistor_SMD:R_0402_1005Metric, symbol Device:R
- removed R54, R55: 1K, Resistor_SMD:R_0402_1005Metric, symbol Device:R
- removed R6: 330Ω, PCM_JLCPCB:R_0402, symbol PCM_JLCPCB-Resistors:0402,330Ω
- removed U4: STLQ015M33R, LoRa_library:SOT-23-5_L3.0-W1.7-P0.95-LS2.8-BR, symbol LoRa_library:STLQ015M33R
- added C10, C15, C16, C18, C3, C32, C33, C39, C40: 100nF, PCM_JLCPCB:C_0402, symbol PCM_JLCPCB-Capacitors:0402,100nF
- added C11, C13, C4: 10uF, PCM_JLCPCB:C_0402, symbol PCM_JLCPCB-Capacitors:0402,10uF
- added C17, C19, C25, C26, C5: 1uF, PCM_JLCPCB:C_0402, symbol PCM_JLCPCB-Capacitors:0402,1uF
- added C22, C37, C38, C49: 12pF, PCM_JLCPCB:C_0402, symbol PCM_JLCPCB-Capacitors:0402,12pF
- added C34, C6: 10uF, PCM_JLCPCB:C_0603, symbol PCM_JLCPCB-Capacitors:0603,10uF,(2)
- added C43: 4.7uF, PCM_JLCPCB:C_0402, symbol PCM_JLCPCB-Capacitors:0402,4.7uF
- added C8: 10nF, PCM_JLCPCB:C_0402, symbol PCM_JLCPCB-Capacitors:0402,10nF
- added C9: 33pF, PCM_JLCPCB:C_0402, symbol PCM_JLCPCB-Capacitors:0402,33pF
- added L4: 24nH, PCM_JLCPCB:L_0402, symbol Device:L
- added R10, R21, R26, R27, R28, R29, R30, R50, R54, R9: 0Ω, PCM_JLCPCB:R_0402, symbol PCM_JLCPCB-Resistors:0402,0Ω
- added R11, R14, R16, R17, R22, R25, R3, R31, R37, R39: 10kΩ, PCM_JLCPCB:R_0402, symbol PCM_JLCPCB-Resistors:0402,10kΩ
- added R12, R19: 470Ω, PCM_JLCPCB:R_0402, symbol PCM_JLCPCB-Resistors:0402,470Ω
- added R13, R42: 5.1kΩ, PCM_JLCPCB:R_0402, symbol PCM_JLCPCB-Resistors:0402,5.1kΩ
- added R18, R2: 1kΩ, PCM_JLCPCB:R_0402, symbol PCM_JLCPCB-Resistors:0402,1kΩ
- added R23, R40: 47kΩ, PCM_JLCPCB:R_0402, symbol PCM_JLCPCB-Resistors:0402,47kΩ
- added R24, R36: 100Ω, PCM_JLCPCB:R_0402, symbol PCM_JLCPCB-Resistors:0402,100Ω
- added R34, R35: 33Ω, PCM_JLCPCB:R_0402, symbol PCM_JLCPCB-Resistors:0402,33Ω
- added U10: XC6206P332MR, PCM_JLCPCB:SOT-23-3_L2.9-W1.6-P1.90-LS2.8-BR, symbol PCM_JLCPCB-Power:LDO, 3.3V, 0.2A
- C12, C14, C31, DNP2, DNP4, DNP6, DNP7: footprint Capacitor_SMD:C_0402_1005Metric -> PCM_JLCPCB:C_0402
- J1: footprint my_footprints:TF-SMD_TF-01A -> LoRa_library:TF-SMD_TF-01A
- L2, L3, L5, L6: footprint Inductor_SMD:L_0402_1005Metric -> PCM_JLCPCB:L_0402
- P1, P2, U15: now left out of the parts list
Connections:
- net +3V3: now also C11.1, C18.1, C19.1, C25.1, C32.1, C33.2, C39.2, C4.1, C8.1, R11.2, R14.2, R16.1, R17.2, R22.1, R25.1, R31.2, R37.2, R39.1
- net +5V: now also C16.1, C34.1, C6.1
- net EN: now also C17.1, R39.2
- net GND: now also C10.1, C11.2, C13.2, C15.2, C16.2, C17.2, C18.2, C19.2, C22.2, C25.2, C26.2, C3.2, C32.2, C33.1, C34.2, C37.1, C38.2, C39.1, C4.2, C40.1, C43.2, C49.2, C5.2, C6.2, C8.2, C9.1, R12.2, R13.2, R19.2, R40.2, R42.2, U10.1 (GND)
- net GPA1: now also R18.2
- net GPB5: now also R2.2
- net GPS_RXD: now also R24.2
- net GPS_TXD: now also R36.2; no longer U1.50 (U0RXD)
- net IO0: now also R22.2
- net IO9/BAT: now also C15.1, R23.2, R40.1
- net LORA_CS: now also R11.1
- net MISOB: now also R14.1, R9.2
- net MTDO/IO40/I2C_SCK: now also R48.2
- net MTMS/IO42/I2C_SDA: now also R47.2
- net SCREEN_CS: now also R37.1
- net SPICLK_N/IO48/SD_CS: now also R17.1
- net SPICS0: now also R3.2
- net SPID: now also R29.2
- net SPIHD: now also R21.2
- net SPIQ: now also R28.2
- net SPISCK: now also R27.2
- net SPIWP: now also R26.2
- net TOUCH_CS: now also R31.1
- net USB_D+: now also R35.2
- net USB_D-: now also R34.2
- net VBAT: now also C13.1, R23.1, U10.3 (VIN)
- net VDD_SPI: now also C26.1, C3.1, R3.1
- net VSYS_SW: now also R50.2
- net XTAL32N: now also C22.1
- net XTAL32P: now also C49.1
- net at J4.9 (Pin_9): now also R9.1
- net at U8.5 (QOD): now also R50.1
- net at C28.1, C29.1, L2.1: now also R54.1
- net at D2.1 (K): now also R12.1
- net at DNP6.1, U18.11 (RF_IN): now also R30.1
- net at U6.4 (I/O2): now also R35.1
- net at U18.14 (VDD_RF): now also R54.2
- net at U1.33 (SPICLK): now also R27.1
- net at U18.6 (V_BCKP): now also C40.2, C43.1, C5.1, C9.2, U10.2 (VOUT)
- net at D4.1 (K): now also R2.1
- net at J3.1 (Pin_1), R20.2: no longer R48.2
- net at D5.1 (K): now also R18.1
- net at DNP2.1, U17.1 (ANT): now also R10.1
- net at U1.31 (SPIWP): now also R26.1
- net at J1.8 (DAT1): now also R16.2
- net at Y2.1: now also C37.2, L4.1
- net at C27.1, DNP7.1: now also R30.2
- net at J1.1 (DAT2): now also R25.2
- net at U1.49 (U0TXD): now also R24.1
- net at DNP4.1, U15.5: now also R10.2
- net at J3.2 (Pin_2), R15.2: no longer R47.2
- net at U1.34 (SPIQ): now also R28.1
- net at L3.2, U1.2 (VDD3P3), U1.3 (VDD3P3): now also C10.2
- net at U1.30 (SPIHD): now also R21.1
- net at U1.35 (SPID): now also R29.1
- net at U1.53 (XTAL_N), Y2.3: now also C38.1
- net at U1.54 (XTAL_P): now also L4.2
- net at U6.6 (I/O1): now also R34.1
- net at U11.A5 (CC1): now also R13.1
- net at U11.B5 (CC2): now also R42.1
- net at D3.1 (K): now also R19.1
- new net: R36.1, U1.50 (U0RXD)
- no-connect marks 26 -> 25
Other:
- moved on the sheet: L3, R15, R20

Commit message: Production ready prototype
Parts:
- added R55, R56, R57, R58, R59, R6, R60, R65: 0Ω, PCM_JLCPCB:R_0402, symbol PCM_JLCPCB-Resistors:0402,0Ω
- added R61, R62, R63, R67: 10kΩ, PCM_JLCPCB:R_0402, symbol PCM_JLCPCB-Resistors:0402,10kΩ
- added TP1: TestPoint, TestPoint:TestPoint_Loop_D1.80mm_Drill1.0mm_Beaded, symbol Connector:TestPoint
Connections:
- net +3V3: now also R61.2, R62.2, R63.2
- net GND: now also R67.2
- net GPB6: now also R61.1
- net LORA_RST: now also U1.23 (GPIO17), R63.1; no longer U14.21 (GPA4)
- net MISOA: now also R58.2, R59.2; no longer J4.13 (Pin_13), U17.13 (MISO)
- net MISOB: now also R60.1; no longer J1.7 (DAT0)
- net MOSIA: now also R57.2; no longer U1.44 (MTCK)
- net MOSIB: now also R6.1; no longer U1.18 (GPIO13)
- net SCKA: now also R56.2; no longer U1.43 (GPIO38)
- net SCKB: now also R55.1; no longer U1.19 (GPIO14)
- net SCREEN_DC: now also R65.2; no longer U1.23 (GPIO17)
- net SCREEN_RST: now also R62.1
- net at U1.52 (GPIO46): now also R65.1, R67.1
- new net: J4.13 (Pin_13), R58.1
- new net: R6.2, U1.18 (GPIO13)
- new net: J1.7 (DAT0), R60.2
- new net: R57.1, U1.44 (MTCK)
- new net: TP1.1, U14.21 (GPA4)
- new net: R55.2, U1.19 (GPIO14)
- new net: R56.1, U1.43 (GPIO38)
- new net: R59.1, U17.13 (MISO)
- no-connect marks 25 -> 24
Other:
- moved on the sheet: AE1, C12, C14, C31, L5, L6, R11
