File: Bare chip/LoRa-device.kicad_pcb (KiCad board)
At the start: 4 copper layers, 86.4 x 50.8 mm, 168 parts, among them J1 Micro_SD_Card_Det1, J3 Conn_01x04_Pin, J4 Conn_01x14_Pin, J6 Conn_01x04_Pin, J8 U.FL, P1 1_25T-1-2A, P2 1_25T-1-2A, SW1 EVQPUC02K, SW2 EVQPUC02K, U1 ESP32-S3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

Commit message: Revised production ready bare chip and module ver.
Parts:
- removed U11: MC-121-L119, LoRa_library:USB-C-SMD_HANBO_MC-121-L119
- added J2: USB_C_Receptacle_USB2.0_14P, Connector_USB:USB_C_Receptacle_HCTL_HC-TYPE-C-16P-01A, F.Cu at (124.7, 122.3)
- J1: footprint LoRa_library:TF-SMD_TF-01A -> Mercurio:TF-SMD_TF-01A
- P1, P2: footprint LoRa_library:CONN-TH_1.25T-1-2A -> Mercurio:CONN-TH_1.25T-1-2A
- SW1, SW2: footprint LoRa_library:SW-SMD_EVQPUD02K -> Mercurio:SW-SMD_EVQPUD02K
- U15: footprint LoRa_library:SMA-SMD_BWSMA-KE-P001 -> Mercurio:SMA-SMD_BWSMA-KE-P001
- U17: footprint LoRa_library:COMM-SMD_17P-L17.0-W16.0-P2.00_RA-01S-P -> Mercurio:COMM-SMD_17P-L17.0-W16.0-P2.00_RA-01S-P
- U18: footprint LoRa_library:GPSM-SMD_18P-L10.1-W9.7-P1.10 -> Mercurio:GPSM-SMD_18P-L10.1-W9.7-P1.10
- U3: footprint LoRa_library:SENSOR-SMD_ICS-43432 -> Mercurio:SENSOR-SMD_ICS-43432
- U5: footprint LoRa_library:SW-TH_SK-12D02-VG5 -> Mercurio:SW-TH_SK-12D02-VG5
- U7: footprint LoRa_library:WSON-10_L2.2-W2.0-P0.40-BL-EP_TI_DLH0010A -> Mercurio:WSON-10_L2.2-W2.0-P0.40-BL-EP_TI_DLH0010A
- U9: footprint LoRa_library:IND-SMD_L4.6-W4.1 -> Mercurio:IND-SMD_L4.6-W4.1
Routing:
- net Net-(J2-D--PadA7): track 4.70 -> 7.50 mm
- net Net-(J2-CC2): track 1.87 -> 4.56 mm
- net Net-(J2-CC1): track 2.17 -> 4.86 mm
- net Net-(J2-D+-PadA6): track 4.89 -> 6.82 mm
- net +5V: track 23.3 -> 25.1 mm
- net VDD_CPU: track 454.1 -> 453.5 mm
- net GND: vias 476 -> 508
