File: Bare chip/LoRa-device.kicad_sch (KiCad schematic)
At the start: 167 parts, among them J1 Micro_SD_Card_Det1, J3 Conn_01x04_Pin, J4 Conn_01x14_Pin, J6 Conn_01x04_Pin, J8 U.FL, P1 1_25T-1-2A, P2 1_25T-1-2A, SW1 EVQPUC02K, SW2 EVQPUC02K, U1 ESP32-S3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

Commit message: Revised production ready bare chip and module ver.
Parts:
- removed U11: MC-121-L119, LoRa_library:USB-C-SMD_HANBO_MC-121-L119, symbol LoRa_library:MC-121-L119
- added J2: USB_C_Receptacle_USB2.0_14P, Connector_USB:USB_C_Receptacle_HCTL_HC-TYPE-C-16P-01A, symbol Connector:USB_C_Receptacle_USB2.0_14P
- DNP2, DNP4, DNP6, DNP7: value ~ -> (none)
- J1: footprint LoRa_library:TF-SMD_TF-01A -> Mercurio:TF-SMD_TF-01A; symbol Connector:Micro_SD_Card_Det1 -> Mercurio:Micro_SD_Card_Det1
- P1, P2: footprint LoRa_library:CONN-TH_1.25T-1-2A -> Mercurio:CONN-TH_1.25T-1-2A; symbol LoRa_library:1_25T-1-2A -> Mercurio:1_25T-1-2A; now in the parts list
- SW1, SW2: footprint LoRa_library:SW-SMD_EVQPUD02K -> Mercurio:SW-SMD_EVQPUD02K; symbol LoRa_library:EVQPUC02K -> Mercurio:EVQPUC02K
- U15: footprint LoRa_library:SMA-SMD_BWSMA-KE-P001 -> Mercurio:SMA-SMD_BWSMA-KE-P001; symbol LoRa_library:HJ-SMA275 -> Mercurio:HJ-SMA275; now in the parts list
- U17: footprint LoRa_library:COMM-SMD_17P-L17.0-W16.0-P2.00_RA-01S-P -> Mercurio:COMM-SMD_17P-L17.0-W16.0-P2.00_RA-01S-P; symbol LoRa_library:RA-01SH-P -> Mercurio:RA-01SH-P
- U18: footprint LoRa_library:GPSM-SMD_18P-L10.1-W9.7-P1.10 -> Mercurio:GPSM-SMD_18P-L10.1-W9.7-P1.10; symbol LoRa_library:L76KB-A58 -> Mercurio:L76KB-A58
- U3: footprint LoRa_library:SENSOR-SMD_ICS-43432 -> Mercurio:SENSOR-SMD_ICS-43432; symbol LoRa_library:ICS-43432 -> Mercurio:ICS-43432
- U5: footprint LoRa_library:SW-TH_SK-12D02-VG5 -> Mercurio:SW-TH_SK-12D02-VG5; symbol LoRa_library:SK-12D02-VG5 -> Mercurio:SK-12D02-VG5
- U7: footprint LoRa_library:WSON-10_L2.2-W2.0-P0.40-BL-EP_TI_DLH0010A -> Mercurio:WSON-10_L2.2-W2.0-P0.40-BL-EP_TI_DLH0010A; symbol LoRa_library:BQ25185DLHR -> Mercurio:BQ25185DLHR
- U9: footprint LoRa_library:IND-SMD_L4.6-W4.1 -> Mercurio:IND-SMD_L4.6-W4.1; symbol LoRa_library:MHCI04020-2R2M-R8 -> Mercurio:MHCI04020-2R2M-R8
Connections:
- net +5V: now also J2.A4 (VBUS), J2.A9 (VBUS), J2.B4 (VBUS), J2.B9 (VBUS)
- net GND: now also J2.A1 (GND), J2.A12 (GND), J2.B1 (GND), J2.B12 (GND), J2.SH (SHIELD)
- net at R13.1: now also J2.A5 (CC1)
- net at U6.3 (I/O2): now also J2.A6 (D+), J2.B6 (D+)
- net at U6.1 (I/O1): now also J2.A7 (D-), J2.B7 (D-)
- net at R42.1: now also J2.B5 (CC2)
- no-connect marks 24 -> 22
Other:
- moved on the sheet: R13, R34, R35, R42, U6
