File: Module/LoRa-device.kicad_pcb (KiCad board)
At the start: 4 copper layers, 86.4 x 50.8 mm, 137 parts, among them J1 Micro_SD_Card_Det1, J2 USB_C_Receptacle_USB2.0_14P, J3 Conn_01x04_Pin, J4 Conn_01x14_Pin, J6 Conn_01x04_Pin, J8 U.FL, P1 1_25T-1-2A, P2 1_25T-1-2A, SW1 EVQPUC02K, SW2 EVQPUC02K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

Commit message: Revised production ready bare chip and module ver.
Parts:
- J1: footprint LoRa_library_modular:TF-SMD_TF-01A -> Mercurio:TF-SMD_TF-01A
- P1, P2: footprint LoRa_library_modular:CONN-TH_1.25T-1-2A -> Mercurio:CONN-TH_1.25T-1-2A
- SW1, SW2: footprint LoRa_library_modular:SW-SMD_EVQPUD02K -> Mercurio:SW-SMD_EVQPUD02K
- U15: footprint LoRa_library_modular:SMA-SMD_BWSMA-KE-P001 -> Mercurio:SMA-SMD_BWSMA-KE-P001
- U17: footprint LoRa_library_modular:COMM-SMD_17P-L17.0-W16.0-P2.00_RA-01S-P -> Mercurio:COMM-SMD_17P-L17.0-W16.0-P2.00_RA-01S-P
- U18: footprint LoRa_library_modular:GPSM-SMD_18P-L10.1-W9.7-P1.10 -> Mercurio:GPSM-SMD_18P-L10.1-W9.7-P1.10
- U3: footprint LoRa_library_modular:SENSOR-SMD_ICS-43432 -> Mercurio:SENSOR-SMD_ICS-43432
- U4: footprint LoRa_library_modular:WIRELM-SMD_ESP32-S3-WROOM-1 -> Mercurio:WIRELM-SMD_ESP32-S3-WROOM-1
- U5: footprint LoRa_library_modular:SW-TH_SK-12D02-VG5 -> Mercurio:SW-TH_SK-12D02-VG5
- U7: footprint LoRa_library_modular:WSON-10_L2.2-W2.0-P0.40-BL-EP_TI_DLH0010A -> Mercurio:WSON-10_L2.2-W2.0-P0.40-BL-EP_TI_DLH0010A
- U9: footprint LoRa_library_modular:IND-SMD_L4.6-W4.1 -> Mercurio:IND-SMD_L4.6-W4.1

Commit message: This version has been sent to production.
Parts:
- removed C55: 10uF, PCM_JLCPCB:C_0603
- removed R66, R68, R69, R9: 0Ω, PCM_JLCPCB:R_0402
- added C37: 10uF, PCM_JLCPCB:C_0603, F.Cu at (116.4, 97.4)
- added R55: 33Ω, PCM_JLCPCB:R_0402, F.Cu at (109.0, 84.9)
- added R56: 33Ω, PCM_JLCPCB:R_0402, F.Cu at (111.5, 88.7)
- added R57: 33Ω, PCM_JLCPCB:R_0402, F.Cu at (168.8, 102.6)
- added R65: 33Ω, PCM_JLCPCB:R_0402, F.Cu at (132.2, 101.8)
- R58, R59, R60, R64: value 0Ω -> 33Ω
- moved R58 39.1 mm to (140.8, 107.6), turned to -90 degrees
- moved R59 26.5 mm to (141.2, 92.1), turned to -90 degrees
- moved R60 12.9 mm to (141.2, 94.6)
- moved J8 4.35 mm to (184.7, 113.3)
- moved C34 2.35 mm to (119.5, 115.6)
- moved C6 2.35 mm to (120.8, 115.6)
- moved R13 2.32 mm to (123.0, 116.1)
- moved R42 2.32 mm to (126.4, 116.1)
- moved R34 2.32 mm to (124.2, 112.8)
- moved R35 2.32 mm to (125.2, 112.8)
- moved U6 2.32 mm to (124.7, 115.5)
- moved DNP6 2.17 mm to (177.4, 113.8)
- moved R70 2.16 mm to (142.6, 87.0)
- moved R30 2.15 mm to (179.0, 113.3)
- moved C27 2.05 mm to (182.1, 113.3)
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Connections:
- R58 pad 1: Net-(J4-Pin_13) -> MISOB
- R58 pad 2: MISOA -> Net-(J1-DAT0)
- R59 pad 1: Net-(U17-MISO) -> Net-(U4-IO39)
- R59 pad 2: MISOA -> MOSIA
- R60 pad 1: MISOB -> Net-(U4-IO38)
- R60 pad 2: Net-(J1-DAT0) -> SCKA
Routing:
- net MISOA: track 64.1 -> 77.9 mm
- net VDD_CPU: track 338.9 -> 342.6 mm
- net Net-(J2-CC1): track 4.81 -> 2.18 mm
- net Net-(J2-CC2): track 4.60 -> 2.00 mm
- net Net-(J2-D--PadA7): track 7.55 -> 5.07 mm
- net USB_D-: track 18.7 -> 21.0 mm
- net USB_D+: track 17.6 -> 19.9 mm
- net Net-(U4-TXD0): track 1.67 -> 3.82 mm
- net GPS_RXD: track 44.9 -> 43.1 mm
- net Net-(J2-D+-PadA6): track 6.84 -> 5.14 mm
- net GPS_TXD: track 42.0 -> 40.6 mm
- net Net-(U4-RXD0): track 1.56 -> 2.89 mm
- net +5V: track 26.8 -> 25.5 mm
- net Net-(U18-RF_IN): track 5.16 -> 3.97 mm
- net Net-(U17-MISO): track 3.62 -> 2.51 mm
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