File: Module/LoRa-device.kicad_sch (KiCad schematic)
At the start: 136 parts, among them J1 Micro_SD_Card_Det1, J2 USB_C_Receptacle_USB2.0_14P, J3 Conn_01x04_Pin, J4 Conn_01x14_Pin, J6 Conn_01x04_Pin, J8 U.FL, P1 1_25T-1-2A, P2 1_25T-1-2A, SW1 EVQPUC02K, SW2 EVQPUC02K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

Commit message: Revised production ready bare chip and module ver.
Parts:
- J1: footprint LoRa_library_modular:TF-SMD_TF-01A -> Mercurio:TF-SMD_TF-01A; symbol Connector:Micro_SD_Card_Det1 -> Mercurio:Micro_SD_Card_Det1
- P1, P2: footprint LoRa_library_modular:CONN-TH_1.25T-1-2A -> Mercurio:CONN-TH_1.25T-1-2A; symbol LoRa_library:1_25T-1-2A -> Mercurio:1_25T-1-2A; now in the parts list
- SW1, SW2: footprint LoRa_library_modular:SW-SMD_EVQPUD02K -> Mercurio:SW-SMD_EVQPUD02K; symbol LoRa_library:EVQPUC02K -> Mercurio:EVQPUC02K
- U15: footprint LoRa_library_modular:SMA-SMD_BWSMA-KE-P001 -> Mercurio:SMA-SMD_BWSMA-KE-P001; symbol LoRa_library:HJ-SMA275 -> Mercurio:HJ-SMA275; now in the parts list
- U17: footprint LoRa_library_modular:COMM-SMD_17P-L17.0-W16.0-P2.00_RA-01S-P -> Mercurio:COMM-SMD_17P-L17.0-W16.0-P2.00_RA-01S-P; symbol LoRa_library:RA-01SH-P -> Mercurio:RA-01SH-P
- U18: footprint LoRa_library_modular:GPSM-SMD_18P-L10.1-W9.7-P1.10 -> Mercurio:GPSM-SMD_18P-L10.1-W9.7-P1.10; symbol LoRa_library:L76KB-A58 -> Mercurio:L76KB-A58
- U3: footprint LoRa_library_modular:SENSOR-SMD_ICS-43432 -> Mercurio:SENSOR-SMD_ICS-43432; symbol LoRa_library:ICS-43432 -> Mercurio:ICS-43432
- U4: footprint LoRa_library_modular:WIRELM-SMD_ESP32-S3-WROOM-1 -> Mercurio:WIRELM-SMD_ESP32-S3-WROOM-1; symbol LoRa_library_modular:ESP32-S3-WROOM-1(N16R8) -> Mercurio:ESP32-S3-WROOM-1(N16R8); now in the parts list
- U5: footprint LoRa_library_modular:SW-TH_SK-12D02-VG5 -> Mercurio:SW-TH_SK-12D02-VG5; symbol LoRa_library:SK-12D02-VG5 -> Mercurio:SK-12D02-VG5
- U7: footprint LoRa_library_modular:WSON-10_L2.2-W2.0-P0.40-BL-EP_TI_DLH0010A -> Mercurio:WSON-10_L2.2-W2.0-P0.40-BL-EP_TI_DLH0010A; symbol LoRa_library:BQ25185DLHR -> Mercurio:BQ25185DLHR
- U9: footprint LoRa_library_modular:IND-SMD_L4.6-W4.1 -> Mercurio:IND-SMD_L4.6-W4.1
Changed lines of the file:
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@@
 	)
 	(junction
-		(at 398.78 182.88)
-		(diameter 0)
-		(color 0 0 0 0)
-	)
-	(junction
 		(at 203.2 248.92)
 		(diameter 0)
@@
 	)
 	(symbol
-		(lib_id "LoRa_library:SK-12D02-VG5")
+		(lib_id "Mercurio:SK-12D02-VG5")
 		(at 365.76 238.76 0)
 		(unit 1)
@@
 			)
 		)
-		(property "Footprint" "LoRa_library_modular:SW-TH_SK-12D02-VG5"
+		(property "Footprint" "Mercurio:SW-TH_SK-12D02-VG5"
 			(at 365.76 248.92 0)
 			(hide yes)
@@
 	)
 	(symbol
-		(lib_id "Connector:Micro_SD_Card_Det1")
+		(lib_id "Mercurio:Micro_SD_Card_Det1")
 		(at 414.02 50.8 0)
 		(unit 1)
@@
 			)
 		)
-		(property "Footprint" "LoRa_library_modular:TF-SMD_TF-01A"
+		(property "Footprint" "Mercurio:TF-SMD_TF-01A"
 			(at 466.09 33.02 0)
 			(hide yes)
@@
 	)
 	(symbol
-		(lib_id "LoRa_library:L76KB-A58")
+		(lib_id "Mercurio:L76KB-A58")
 		(at 52.07 153.67 0)
 		(unit 1)
@@
 			)
 		)
-		(property "Footprint" "LoRa_library_modular:GPSM-SMD_18P-L10.1-W9.7-P1.10"
+		(property "Footprint" "Mercurio:GPSM-SMD_18P-L10.1-W9.7-P1.10"
 			(at 52.07 163.83 0)
 			(hide yes)
@@
 			)
 		)
-		(property "Footprint" "LoRa_library_modular:IND-SMD_L4.6-W4.1"
+		(property "Footprint" "Mercurio:IND-SMD_L4.6-W4.1"
 			(at 149.86 257.81 0)
 			(hide yes)
@@
 	)
 	(symbol
-		(lib_id "LoRa_library:1_25T-1-2A")
+		(lib_id "Mercurio:1_25T-1-2A")
 		(at 250.19 274.32 0)
 		(unit 1)
 		(body_style 1)
 		(exclude_from_sim no)
-		(in_bom no)
+		(in_bom yes)
 		(on_board yes)
 		(in_pos_files yes)
@@
 			)
 		)
-		(property "Footprint" "LoRa_library_modular:CONN-TH_1.25T-1-2A"
+		(property "Footprint" "Mercurio:CONN-TH_1.25T-1-2A"
 			(at 250.19 284.48 0)
 			(hide yes)
@@
 	)
 	(symbol
-		(lib_id "LoRa_library:1_25T-1-2A")
+		(lib_id "Mercurio:1_25T-1-2A")
 		(at 339.09 204.47 180)
 		(unit 1)
 		(body_style 1)
 		(exclude_from_sim no)
-		(in_bom no)
+		(in_bom yes)
 		(on_board yes)
 		(in_pos_files yes)
@@
 			)
 		)
-		(property "Footprint" "LoRa_library_modular:CONN-TH_1.25T-1-2A"
+		(property "Footprint" "Mercurio:CONN-TH_1.25T-1-2A"
 			(at 339.09 194.31 0)
 			(hide yes)
@@
 	)
 	(symbol
-		(lib_id "LoRa_library_modular:ESP32-S3-WROOM-1(N16R8)")
+		(lib_id "Mercurio:ESP32-S3-WROOM-1(N16R8)")
 		(at 219.71 129.54 0)
 		(unit 1)
 		(body_style 1)
 		(exclude_from_sim no)
-		(in_bom no)
+		(in_bom yes)
 		(on_board yes)
 		(in_pos_files yes)
@@
 			)
 		)
-		(property "Footprint" "LoRa_library_modular:WIRELM-SMD_ESP32-S3-WROOM-1"
+		(property "Footprint" "Mercurio:WIRELM-SMD_ESP32-S3-WROOM-1"
 			(at 219.71 139.7 0)
 			(hide yes)
@@
 	)
 	(symbol
-		(lib_id "LoRa_library:HJ-SMA275")
+		(lib_id "Mercurio:HJ-SMA275")
 		(at 113.03 86.36 90)
 		(unit 1)
 		(body_style 1)
 		(exclude_from_sim no)
-		(in_bom no)
+		(in_bom yes)
 		(on_board yes)
 		(in_pos_files yes)
@@
 			)
 		)
-		(property "Footprint" "LoRa_library_modular:SMA-SMD_BWSMA-KE-P001"
+		(property "Footprint" "Mercurio:SMA-SMD_BWSMA-KE-P001"
 			(at 123.19 86.36 0)
 			(hide yes)
@@
 	)
 	(symbol
-		(lib_id "LoRa_library:EVQPUC02K")
+		(lib_id "Mercurio:EVQPUC02K")
 		(at 104.14 40.64 0)
 		(unit 1)
@@
 			)
 		)
-		(property "Footprint" "LoRa_library_modular:SW-SMD_EVQPUD02K"
+		(property "Footprint" "Mercurio:SW-SMD_EVQPUD02K"
 			(at 104.14 50.8 0)
 			(hide yes)
@@
 	)
 	(symbol
-		(lib_id "LoRa_library:RA-01SH-P")
+		(lib_id "Mercurio:RA-01SH-P")
 		(at 50.8 88.9 0)
 		(unit 1)
@@
 		(fields_autoplaced yes)
 		(property "Reference" "U17"
-			(at 50.8 71.12 0)
+			(at 50.8 104.14 0)
 			(show_name no)
 			(do_not_autoplace no)
@@
 		)
 		(property "Value" "RA-01SH-P"
-			(at 50.8 73.66 0)
+			(at 50.8 106.68 0)
 			(show_name no)
 			(do_not_autoplace no)
@@
 			)
 		)
-		(property "Footprint" "LoRa_library_modular:COMM-SMD_17P-L17.0-W16.0-P2.00_RA-01S-P"
+		(property "Footprint" "Mercurio:COMM-SMD_17P-L17.0-W16.0-P2.00_RA-01S-P"
 			(at 51.054 104.14 0)
 			(hide yes)
@@
 	)
 	(symbol
-		(lib_id "LoRa_library:ICS-43432")
+		(lib_id "Mercurio:ICS-43432")
 		(at 398.78 191.77 0)
 		(unit 1)
@@
 			)
 		)
-		(property "Footprint" "LoRa_library_modular:SENSOR-SMD_ICS-43432"
+		(property "Footprint" "Mercurio:SENSOR-SMD_ICS-43432"
 			(at 398.78 201.93 0)
 			(hide yes)
@@
 	)
 	(symbol
-		(lib_id "LoRa_library:EVQPUC02K")
+		(lib_id "Mercurio:EVQPUC02K")
 		(at 127 33.02 0)
 		(unit 1)
@@
 			)
 		)
-		(property "Footprint" "LoRa_library_modular:SW-SMD_EVQPUD02K"
+		(property "Footprint" "Mercurio:SW-SMD_EVQPUD02K"
 			(at 127 43.18 0)
 			(hide yes)
@@
 	)
 	(symbol
-		(lib_id "LoRa_library:BQ25185DLHR")
+		(lib_id "Mercurio:BQ25185DLHR")
 		(at 247.65 248.92 0)
 		(unit 1)
@@
 			)
 		)
-		(property "Footprint" "LoRa_library_modular:WSON-10_L2.2-W2.0-P0.40-BL-EP_TI_DLH0010A"
+		(property "Footprint" "Mercurio:WSON-10_L2.2-W2.0-P0.40-BL-EP_TI_DLH0010A"
 			(at 247.65 259.08 0)
 			(hide yes)

Commit message: This version has been sent to production.
Parts:
- removed C55: 10uF, PCM_JLCPCB:C_0603, symbol PCM_JLCPCB-Capacitors:0603,10uF
- removed R58, R59, R60, R64, R66, R68, R69, R9: 0Ω, PCM_JLCPCB:R_0402, symbol PCM_JLCPCB-Resistors:0402,0Ω
- added C37: 10uF, PCM_JLCPCB:C_0603, symbol PCM_JLCPCB-Capacitors:0603,10uF,(2)
- added R55, R56, R57, R58, R59, R60, R64, R65: 33Ω, PCM_JLCPCB:R_0402, symbol PCM_JLCPCB-Resistors:0402,33Ω
- D2, D4, D5: MNF PART NUMBER C2286 -> (none); Part (none) -> KT-0603R
- DNP2, DNP4, DNP6, DNP7, J3, J4, J6, P1, P2: now left out of the parts list
- J1: Part (none) -> TF-01A
- J2: Part (none) -> HC-TYPE-C-16P-3M2S
- J8: Part (none) -> BWU.FL-IPEX1
- L2: MNF PART NUMBER C32836 -> (none); Part (none) -> SDCL1005C68NJTDF
- SW1, SW2: Part (none) -> EVQPUC02K
- U12: Part (none) -> TLV62569DBVR
- U14: Part (none) -> MCP23017T-E/ML
- U15: Part (none) -> HJ-SMA275; now left out of the parts list
- U17: Part (none) -> Ra-01SH-P
- U18: Part (none) -> L76KB-A58
- U19: Part (none) -> MAX98357AETE+T
- U3: Part (none) -> ICS-43432
- U4: Part (none) -> ESP32-S3-WROOM-1(N16R8)
- U5: Part (none) -> SK-12D02-VG5
- U6: Part (none) -> USBLC6-2P6
- U7: Part (none) -> BQ25185DLHR
- U8: MNF PART NUMBER C3235537 -> (none); Part (none) -> TPS22917LDBVR
- U9: Part (none) -> MHCI04020-2R2M-R8
Connections:
- net +3V3: now also C37.1
- net GND: now also C37.2
- net MISOA: now also R55.1, R57.2
- net MISOB: now also R56.1, R58.1
- net MOSIA: now also R59.2
- net MOSIB: now also R64.1
- net SCKA: now also R60.2
- net SCKB: now also R65.1
- net at J4.13 (Pin_13): now also R55.2
- net at J4.9 (Pin_9): now also R56.2
- net at U4.32 (IO39): now also R59.1
- net at J1.7 (DAT0): now also R58.2
- net at U4.31 (IO38): now also R60.1
- net at U17.13 (MISO): now also R57.1
- net at U4.21 (IO13): now also R64.2
- net at U4.22 (IO14): now also R65.2
